File: tutorial.kicad_pcb (KiCad board)
At the start: 2 copper layers, 284.5 x 94 mm, 129 parts, among them SW0:0 CTRL, SW0:1 SUPER, SW0:10 ALT, SW0:11 MENU, SW0:12 SUPER, SW0:13 CTRL, SW0:2 ALT, SW0:4 SPACE, SW1:1 SHIFT, SW1:10 ., SW1:11 ?, SW1:12 SHIFT, SW1:2 Z, SW1:3 X, SW1:4 C, SW1:5 V, SW1:6 B, SW1:7 N, SW1:8 M, SW1:9 ,, SW2:0 CAPS, SW2:1 A, SW2:10 ;, SW2:11 ', SW2:12 ENTER, SW2:2 S, SW2:3 D, SW2:4 F, SW2:5 G, SW2:6 H, SW2:7 J, SW2:8 K, SW2:9 L, SW3:0 TAB, SW3:1 Q, SW3:10 P, SW3:11 {, SW3:12 }, SW3:13 BCKSL, SW3:2 W, SW3:3 E, SW3:4 R, SW3:5 T, SW3:6 Y, SW3:7 U, SW3:8 I, SW3:9 O, SW4:0 TILDE, SW4:1 1, SW4:10 0, SW4:11 -, SW4:12 =, SW4:13 BCKSP, SW4:2 2, SW4:3 3, SW4:4 4, SW4:5 5, SW4:6 6, SW4:7 7, SW4:8 8, SW4:9 9, U1 TEENSY2.0

Commit message: first commit
Parts:
- removed the SW4:2 at (88.9, 50.8)
- added D0:14: D, footprints:DIODE, F.Cu at (399.0, 153.0)
- added D0:15: D, footprints:DIODE, F.Cu at (421.5, 153.0)
- added D0:3: D, footprints:DIODE, F.Cu at (139.5, 153.0)
- added D0:5: D, footprints:DIODE, F.Cu at (183.0, 153.0)
- added D0:6: D, footprints:DIODE, F.Cu at (205.0, 153.0)
- added D0:7: D, footprints:DIODE, F.Cu at (227.0, 153.0)
- added D0:8: D, footprints:DIODE, F.Cu at (249.0, 153.0)
- added D0:9: D, footprints:DIODE, F.Cu at (271.5, 153.0)
- added D1:0: D, footprints:DIODE, F.Cu at (443.5, 153.0)
- added D1:13: D, footprints:DIODE, F.Cu at (341.5, 175.0)
- added D1:14: D, footprints:DIODE, F.Cu at (369.0, 175.0)
- added D1:15: D, footprints:DIODE, F.Cu at (399.5, 175.0)
- added D2:13: D, footprints:DIODE, F.Cu at (325.5, 197.0)
- added D2:14: D, footprints:DIODE, F.Cu at (362.5, 197.0)
- added D2:15: D, footprints:DIODE, F.Cu at (407.5, 228.5)
- added D3:14: D, footprints:DIODE, F.Cu at (429.5, 228.5)
- added D3:15: D, footprints:DIODE, F.Cu at (86.5, 228.5)
- added D4:14: D, footprints:DIODE, F.Cu at (491.5, 197.0)
- added D4:15: D, footprints:DIODE, F.Cu at (513.5, 197.0)
- added D5:0: D, footprints:DIODE, F.Cu at (535.5, 186.0)
- added D5:1: D, footprints:DIODE, F.Cu at (469.5, 175.0)
- added D5:10: D, footprints:DIODE, F.Cu at (123.5, 127.0)
- added D5:11: D, footprints:DIODE, F.Cu at (145.5, 127.0)
- added D5:12: D, footprints:DIODE, F.Cu at (167.5, 127.0)
- added D5:13: D, footprints:DIODE, F.Cu at (204.5, 127.0)
- added D5:14: D, footprints:DIODE, F.Cu at (226.5, 127.0)
- added D5:15: D, footprints:DIODE, F.Cu at (248.5, 127.0)
- added D5:2: D, footprints:DIODE, F.Cu at (491.5, 175.0)
- added D5:3: D, footprints:DIODE, F.Cu at (513.5, 175.0)
- added D5:4: D, footprints:DIODE, F.Cu at (469.5, 153.0)
- added D5:5: D, footprints:DIODE, F.Cu at (491.5, 153.0)
- added D5:6: D, footprints:DIODE, F.Cu at (513.5, 153.0)
- added D5:7: D, footprints:DIODE, F.Cu at (534.0, 151.0)
- added D5:8: D, footprints:DIODE, F.Cu at (73.5, 153.0)
- added D5:9: D, footprints:DIODE, F.Cu at (101.5, 127.0)
- added D6:0: D, footprints:DIODE, F.Cu at (270.5, 127.0)
- added D6:1: D, footprints:DIODE, F.Cu at (307.5, 127.0)
- added D6:10: D, footprints:DIODE, F.Cu at (145.5, 105.0)
- added D6:11: D, footprints:DIODE, F.Cu at (167.5, 105.0)
- added D6:12: D, footprints:DIODE, F.Cu at (204.5, 105.0)
- added D6:13: D, footprints:DIODE, F.Cu at (226.5, 105.0)
- added D6:14: D, footprints:DIODE, F.Cu at (248.5, 105.0)
- added D6:15: D, footprints:DIODE, F.Cu at (270.0, 105.0)
- added D6:2: D, footprints:DIODE, F.Cu at (329.5, 127.0)
- added D6:3: D, footprints:DIODE, F.Cu at (351.5, 127.0)
- added D6:4: D, footprints:DIODE, F.Cu at (373.5, 127.0)
- added D6:5: D, footprints:DIODE, F.Cu at (399.5, 127.0)
- added D6:6: D, footprints:DIODE, F.Cu at (421.5, 127.0)
- added D6:7: D, footprints:DIODE, F.Cu at (443.5, 127.0)
- added D6:8: D, footprints:DIODE, F.Cu at (101.5, 105.0)
- added D6:9: D, footprints:DIODE, F.Cu at (123.5, 105.0)
- added D7:0: D, footprints:DIODE, F.Cu at (307.0, 105.0)
- added D7:1: D, footprints:DIODE, F.Cu at (329.0, 105.0)
- added D7:2: D, footprints:DIODE, F.Cu at (351.0, 105.0)
- added D7:3: D, footprints:DIODE, F.Cu at (373.5, 105.0)
- added SW0:14: INS, Keyboard:CHERRY_PCB_100H_With_led2, F.Cu at (398.0, 142.0)
- added SW0:15: HOME, Keyboard:CHERRY_PCB_100H_With_led2, F.Cu at (420.0, 142.0)
- added SW0:3: 3, Keyboard:CHERRY_PCB_100H_With_led2, F.Cu at (138.0, 142.0)
- added SW0:5: 5, Keyboard:CHERRY_PCB_100H_With_led2, F.Cu at (182.0, 142.0)
- added SW0:6: 6, Keyboard:CHERRY_PCB_100H_With_led2, F.Cu at (204.0, 142.0)
- added SW0:7: 7, Keyboard:CHERRY_PCB_100H_With_led2, F.Cu at (226.0, 142.0)
- added SW0:8: 8, Keyboard:CHERRY_PCB_100H_With_led2, F.Cu at (248.0, 142.0)
- added SW0:9: 9, Keyboard:CHERRY_PCB_100H_With_led2, F.Cu at (270.0, 142.0)
- added SW1:0: PAGE_UP, Keyboard:CHERRY_PCB_100H_With_led2, F.Cu at (442.0, 142.0)
- added SW1:13: ], Keyboard:CHERRY_PCB_100H_With_led2, F.Cu at (340.0, 164.0)
- added SW1:14: \, Keyboard:CHERRY_PCB_100H_With_led2, F.Cu at (367.0, 164.0)
- added SW1:15: DEL, Keyboard:CHERRY_PCB_100H_With_led2, F.Cu at (398.0, 164.0)
- added SW2:13: `, Keyboard:CHERRY_PCB_100H_With_led2, F.Cu at (324.0, 186.0)
- added SW2:14: ENTER, Keyboard:CHERRY_PCB_100H_With_led2, F.Cu at (361.0, 186.0)
- added SW2:15: LEFT, Keyboard:CHERRY_PCB_100H_With_led2, F.Cu at (398.0, 230.0)
- added SW3:14: DOWN, Keyboard:CHERRY_PCB_100H_With_led2, F.Cu at (420.0, 230.0)
- added SW3:15: L_CTRL, Keyboard:CHERRY_PCB_100H_With_led2, F.Cu at (77.0, 230.0)
- added SW4:14: KEYPAD_5, Keyboard:CHERRY_PCB_100H_With_led2, F.Cu at (490.0, 186.0)
- added SW4:15: KEYPAD_6, Keyboard:CHERRY_PCB_100H_With_led2, F.Cu at (512.0, 186.0)
- added SW4:2 (x2): SPACE, Keyboard:CHERRY_PCB_100H_With_led2, F.Cu at (205.5, 230.0)
- added SW5:0: KEYPAD_+, Keyboard:CHERRY_PCB_100H_With_led2, F.Cu at (534.0, 175.0)
- added SW5:1: KEYPAD_7, Keyboard:CHERRY_PCB_100H_With_led2, F.Cu at (468.0, 164.0)
- added SW5:10: F2, Keyboard:CHERRY_PCB_100H_With_led2, F.Cu at (122.0, 116.0)
- added SW5:11: F3, Keyboard:CHERRY_PCB_100H_With_led2, F.Cu at (144.0, 116.0)
- added SW5:12: F4, Keyboard:CHERRY_PCB_100H_With_led2, F.Cu at (166.0, 116.0)
- added SW5:13: F5, Keyboard:CHERRY_PCB_100H_With_led2, F.Cu at (203.0, 116.0)
- added SW5:14: F6, Keyboard:CHERRY_PCB_100H_With_led2, F.Cu at (225.0, 116.0)
- added SW5:15: F7, Keyboard:CHERRY_PCB_100H_With_led2, F.Cu at (247.0, 116.0)
- added SW5:2: KEYPAD_8, Keyboard:CHERRY_PCB_100H_With_led2, F.Cu at (490.0, 164.0)
- added SW5:3: KEYPAD_9, Keyboard:CHERRY_PCB_100H_With_led2, F.Cu at (512.0, 164.0)
- added SW5:4: KEYPAD_NUMLOCK, Keyboard:CHERRY_PCB_100H_With_led2, F.Cu at (468.0, 142.0)
- added SW5:5: KEYPAD_/, Keyboard:CHERRY_PCB_100H_With_led2, F.Cu at (490.0, 142.0)
- added SW5:6: KEYPAD_*, Keyboard:CHERRY_PCB_100H_With_led2, F.Cu at (512.0, 142.0)
- added SW5:7: KEIPAD_-, Keyboard:CHERRY_PCB_100H_With_led2, F.Cu at (534.0, 142.0)
- added SW5:8: TILDE, Keyboard:CHERRY_PCB_100H_With_led2, F.Cu at (72.0, 142.0)
- added SW5:9: F1, Keyboard:CHERRY_PCB_100H_With_led2, F.Cu at (100.0, 116.0)
- added SW6:0: F8, Keyboard:CHERRY_PCB_100H_With_led2, F.Cu at (269.0, 116.0)
- added SW6:1: F9, Keyboard:CHERRY_PCB_100H_With_led2, F.Cu at (306.0, 116.0)
- added SW6:10: K3, Keyboard:CHERRY_PCB_100H_With_led2, F.Cu at (144.0, 94.0)
- added SW6:11: K4, Keyboard:CHERRY_PCB_100H_With_led2, F.Cu at (166.0, 94.0)
- added SW6:12: K5, Keyboard:CHERRY_PCB_100H_With_led2, F.Cu at (203.0, 94.0)
- added SW6:13: K6, Keyboard:CHERRY_PCB_100H_With_led2, F.Cu at (225.0, 94.0)
- added SW6:14: K7, Keyboard:CHERRY_PCB_100H_With_led2, F.Cu at (247.0, 94.0)
- added SW6:15: K8, Keyboard:CHERRY_PCB_100H_With_led2, F.Cu at (269.0, 94.0)
- added SW6:2: F10, Keyboard:CHERRY_PCB_100H_With_led2, F.Cu at (328.0, 116.0)
- added SW6:3: F11, Keyboard:CHERRY_PCB_100H_With_led2, F.Cu at (350.0, 116.0)
- added SW6:4: F12, Keyboard:CHERRY_PCB_100H_With_led2, F.Cu at (372.0, 116.0)
- added SW6:5: PRINTSCREEN, Keyboard:CHERRY_PCB_100H_With_led2, F.Cu at (398.0, 116.0)
- added SW6:6: SCROLL_LOCK, Keyboard:CHERRY_PCB_100H_With_led2, F.Cu at (420.0, 116.0)
- added SW6:7: PAUSE, Keyboard:CHERRY_PCB_100H_With_led2, F.Cu at (442.0, 116.0)
- added SW6:8: K1, Keyboard:CHERRY_PCB_100H_With_led2, F.Cu at (100.0, 94.0)
- added SW6:9: K2, Keyboard:CHERRY_PCB_100H_With_led2, F.Cu at (122.0, 94.0)
- added SW7:0: K9, Keyboard:CHERRY_PCB_100H_With_led2, F.Cu at (306.0, 94.0)
- added SW7:1: K10, Keyboard:CHERRY_PCB_100H_With_led2, F.Cu at (328.0, 94.0)
- added SW7:2: K11, Keyboard:CHERRY_PCB_100H_With_led2, F.Cu at (350.0, 94.0)
- added SW7:3: K12, Keyboard:CHERRY_PCB_100H_With_led2, F.Cu at (372.0, 94.0)
- added SW7:4: Fake1, Keyboard:CHERRY_PCB_100H_With_led2, F.Cu at (235.0, 230.0)
- added SW7:5: Fake2, Keyboard:CHERRY_PCB_100H_With_led2, F.Cu at (175.5, 230.5)
- SW0:0: value CTRL -> ESC; footprint footprints:CHERRY_PCB_125H -> Keyboard:CHERRY_PCB_100H_With_led2
- SW0:1: value SUPER -> 1; footprint footprints:CHERRY_PCB_125H -> Keyboard:CHERRY_PCB_100H_With_led2
- SW0:10: value ALT -> 0; footprint footprints:CHERRY_PCB_125H -> Keyboard:CHERRY_PCB_100H_With_led2
- SW0:11: value MENU -> -; footprint footprints:CHERRY_PCB_125H -> Keyboard:CHERRY_PCB_100H_With_led2
- SW0:12: value SUPER -> =; footprint footprints:CHERRY_PCB_125H -> Keyboard:CHERRY_PCB_100H_With_led2
- SW0:13: value CTRL -> BCKSPC; footprint footprints:CHERRY_PCB_125H -> Keyboard:CHERRY_PCB_100H_With_led2
- SW0:2: value ALT -> 2; footprint footprints:CHERRY_PCB_125H -> Keyboard:CHERRY_PCB_100H_With_led2
- SW0:4: value SPACE -> 4; footprint footprints:CHERRY_PCB_625H -> Keyboard:CHERRY_PCB_100H_With_led2
- SW1:1: value SHIFT -> TAB; footprint footprints:CHERRY_PCB_225H -> Keyboard:CHERRY_PCB_100H_With_led2
- SW1:10: value . -> O; footprint footprints:CHERRY_PCB_100H -> Keyboard:CHERRY_PCB_100H_With_led2
- SW1:11: value ? -> P; footprint footprints:CHERRY_PCB_100H -> Keyboard:CHERRY_PCB_100H_With_led2
- SW1:12: value SHIFT -> [; footprint footprints:CHERRY_PCB_275H -> Keyboard:CHERRY_PCB_100H_With_led2
- SW1:2: value Z -> Q; footprint footprints:CHERRY_PCB_100H -> Keyboard:CHERRY_PCB_100H_With_led2
- SW1:3: value X -> W; footprint footprints:CHERRY_PCB_100H -> Keyboard:CHERRY_PCB_100H_With_led2
- SW1:4: value C -> E; footprint footprints:CHERRY_PCB_100H -> Keyboard:CHERRY_PCB_100H_With_led2
- SW1:5: value V -> R; footprint footprints:CHERRY_PCB_100H -> Keyboard:CHERRY_PCB_100H_With_led2
- SW1:6: value B -> T; footprint footprints:CHERRY_PCB_100H -> Keyboard:CHERRY_PCB_100H_With_led2
- SW1:7: value N -> Y; footprint footprints:CHERRY_PCB_100H -> Keyboard:CHERRY_PCB_100H_With_led2
- SW1:8: value M -> U; footprint footprints:CHERRY_PCB_100H -> Keyboard:CHERRY_PCB_100H_With_led2
- SW1:9: value , -> I; footprint footprints:CHERRY_PCB_100H -> Keyboard:CHERRY_PCB_100H_With_led2
- SW2:0: value CAPS -> END; footprint footprints:CHERRY_PCB_175H -> Keyboard:CHERRY_PCB_100H_With_led2
- SW2:1: value A -> PAGE_DOWN; footprint footprints:CHERRY_PCB_100H -> Keyboard:CHERRY_PCB_100H_With_led2
- SW2:10: value ; -> K; footprint footprints:CHERRY_PCB_100H -> Keyboard:CHERRY_PCB_100H_With_led2
- SW2:11: value ' -> L; footprint footprints:CHERRY_PCB_100H -> Keyboard:CHERRY_PCB_100H_With_led2
- SW2:12: value ENTER -> ;; footprint footprints:CHERRY_PCB_225H -> Keyboard:CHERRY_PCB_100H_With_led2
- SW2:2: value S -> CAPSLOCK; footprint footprints:CHERRY_PCB_100H -> Keyboard:CHERRY_PCB_100H_With_led2
- SW2:3: value D -> A; footprint footprints:CHERRY_PCB_100H -> Keyboard:CHERRY_PCB_100H_With_led2
- SW2:4: value F -> S; footprint footprints:CHERRY_PCB_100H -> Keyboard:CHERRY_PCB_100H_With_led2
- SW2:5: value G -> D; footprint footprints:CHERRY_PCB_100H -> Keyboard:CHERRY_PCB_100H_With_led2
- SW2:6: value H -> F; footprint footprints:CHERRY_PCB_100H -> Keyboard:CHERRY_PCB_100H_With_led2
- SW2:7: value J -> G; footprint footprints:CHERRY_PCB_100H -> Keyboard:CHERRY_PCB_100H_With_led2
- SW2:8: value K -> H; footprint footprints:CHERRY_PCB_100H -> Keyboard:CHERRY_PCB_100H_With_led2
- SW2:9: value L -> J; footprint footprints:CHERRY_PCB_100H -> Keyboard:CHERRY_PCB_100H_With_led2
- SW3:0: value TAB -> RIGHT; footprint footprints:CHERRY_PCB_150H -> Keyboard:CHERRY_PCB_100H_With_led2
- SW3:1: value Q -> L_SHIFT; footprint footprints:CHERRY_PCB_100H -> Keyboard:CHERRY_PCB_100H_With_led2
- SW3:10: value P -> .; footprint footprints:CHERRY_PCB_100H -> Keyboard:CHERRY_PCB_100H_With_led2
- SW3:11: value { -> /; footprint footprints:CHERRY_PCB_100H -> Keyboard:CHERRY_PCB_100H_With_led2
- SW3:12: value } -> R_SHIFT; footprint footprints:CHERRY_PCB_100H -> Keyboard:CHERRY_PCB_100H_With_led2
- SW3:13: value BCKSL -> UP; footprint footprints:CHERRY_PCB_150H -> Keyboard:CHERRY_PCB_100H_With_led2
- SW3:2: value W -> Z; footprint footprints:CHERRY_PCB_100H -> Keyboard:CHERRY_PCB_100H_With_led2
- SW3:3: value E -> X; footprint footprints:CHERRY_PCB_100H -> Keyboard:CHERRY_PCB_100H_With_led2
- SW3:4: value R -> C; footprint footprints:CHERRY_PCB_100H -> Keyboard:CHERRY_PCB_100H_With_led2
- SW3:5: value T -> V; footprint footprints:CHERRY_PCB_100H -> Keyboard:CHERRY_PCB_100H_With_led2
- SW3:6: value Y -> B; footprint footprints:CHERRY_PCB_100H -> Keyboard:CHERRY_PCB_100H_With_led2
- SW3:7: value U -> N; footprint footprints:CHERRY_PCB_100H -> Keyboard:CHERRY_PCB_100H_With_led2
- SW3:8: value I -> M; footprint footprints:CHERRY_PCB_100H -> Keyboard:CHERRY_PCB_100H_With_led2
- SW3:9: value O -> ,; footprint footprints:CHERRY_PCB_100H -> Keyboard:CHERRY_PCB_100H_With_led2
- SW4:0: value TILDE -> L_SUPER; footprint footprints:CHERRY_PCB_100H -> Keyboard:CHERRY_PCB_100H_With_led2
- SW4:1: value 1 -> L_ALT; footprint footprints:CHERRY_PCB_100H -> Keyboard:CHERRY_PCB_100H_With_led2
- SW4:10: value 0 -> KEYPAD_1; footprint footprints:CHERRY_PCB_100H -> Keyboard:CHERRY_PCB_100H_With_led2
- SW4:11: value - -> KEYPAD_2; footprint footprints:CHERRY_PCB_100H -> Keyboard:CHERRY_PCB_100H_With_led2
- SW4:12: value = -> KEYPAD_3; footprint footprints:CHERRY_PCB_100H -> Keyboard:CHERRY_PCB_100H_With_led2
- SW4:13: value BCKSP -> KEYPAD_4; footprint footprints:CHERRY_PCB_200H -> Keyboard:CHERRY_PCB_100H_With_led2
- SW4:3: value 3 -> R_ALT; footprint footprints:CHERRY_PCB_100H -> Keyboard:CHERRY_PCB_100H_With_led2
- SW4:4: value 4 -> R_SUPER; footprint footprints:CHERRY_PCB_100H -> Keyboard:CHERRY_PCB_100H_With_led2
- SW4:5: value 5 -> MENU; footprint footprints:CHERRY_PCB_100H -> Keyboard:CHERRY_PCB_100H_With_led2
- SW4:6: value 6 -> R_CTRL; footprint footprints:CHERRY_PCB_100H -> Keyboard:CHERRY_PCB_100H_With_led2
- SW4:7: value 7 -> KEYPAD_0; footprint footprints:CHERRY_PCB_100H -> Keyboard:CHERRY_PCB_100H_With_led2
- SW4:8: value 8 -> KEYPAD_DEL; footprint footprints:CHERRY_PCB_100H -> Keyboard:CHERRY_PCB_100H_With_led2
- SW4:9: value 9 -> KEYPAD_ENTER; footprint footprints:CHERRY_PCB_100H -> Keyboard:CHERRY_PCB_100H_With_led2
- U1: value TEENSY2.0 -> Teensy3.2; footprint footprints:TEENSY_2.0 -> Teensy:Teensy30_31_32_LC
- moved U1 492.4 mm to (512.0, 99.5), turned to 180 degrees
- moved R2 434.9 mm to (492.5, 115.0)
- moved L2 432.1 mm to (489.0, 118.5)
- moved D3:0 418.6 mm to (451.5, 228.0)
- moved SW3:0 418.3 mm to (442.0, 230.0)
- moved D2:1 377.6 mm to (443.5, 175.0), turned to 0 degrees
- moved D4:8 371.8 mm to (521.5, 228.5)
- moved SW2:0 369.8 mm to (420.0, 164.0)
- moved D4:9 366.7 mm to (535.0, 228.0), turned to 0 degrees
- moved SW2:1 365.7 mm to (442.0, 164.0)
- moved D2:0 365.5 mm to (421.5, 175.0), turned to 0 degrees
- moved D4:7 359.4 mm to (488.5, 228.0)
- moved SW4:8 357.0 mm to (512.0, 230.0)
- moved SW4:9 354.2 mm to (534.0, 219.0)
- moved SW4:7 345.0 mm to (479.0, 230.0)
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Connections:
- D1:12 pad 2: Net-(D1:12-Pad2) -> /COL12
- D2:12 pad 2: Net-(D2:12-Pad2) -> /COL12
- U1 pad 1: GND -> Net-(U1-Pad1)
- U1 pad 10: /ROW4 -> /ROW3
- U1 pad 11: /COL12 -> /COL10
- U1 pad 12: /COL13 -> /COL11
- U1 pad 13: /COL3 -> /COL12
- U1 pad 14: VCC -> /COL13
- U1 pad 15: GND -> Net-(U1-Pad15)
- U1 pad 17: /COL0 -> Net-(U1-Pad17)
- U1 pad 18: /COL1 -> Net-(U1-Pad18)
- U1 pad 19: /COL2 -> Net-(U1-Pad19)
- U1 pad 2: /COL6 -> /COL4
- U1 pad 21: Net-(U1-Pad21) -> /ROW1
- U1 pad 22: Net-(U1-Pad22) -> /COL7
- U1 pad 23: /COL4 -> /COL0
- U1 pad 24: /LED_C -> /COL1
- U1 pad 25: /ROW3 -> /COL3
- U1 pad 26: /ROW2 -> /COL2
- U1 pad 27: /ROW1 -> /ROW5
- U1 pad 28: /ROW0 -> /ROW6
- U1 pad 29: VCC -> /COL8
- U1 pad 3: /COL7 -> /COL5
- U1 pad 30: Net-(U1-Pad30) -> /COL9
- U1 pad 31: /COL5 -> Net-(U1-Pad31)
- U1 pad 4: /COL8 -> /ROW0
- U1 pad 5: /COL9 -> /COL14
- U1 pad 6: /COL10 -> /COL15
- U1 pad 7: /COL11 -> /ROW7
- U1 pad 8: /LED_B -> /ROW4
- U1 pad 9: /LED_A -> /ROW2
Routing:
- net /ROW3: track 292.7 -> 0.00 mm
- net /ROW4: track 291.8 -> 0.00 mm
- net /ROW0: track 286.5 -> 0.00 mm
- net /ROW2: track 279.7 -> 0.00 mm
- net /ROW1: track 266.7 -> 0.00 mm
- net /COL1: track 103.0 -> 0.00 mm
- net /COL4: track 99.6 -> 0.00 mm
- net /COL2: track 98.6 -> 0.00 mm
- net /COL10: track 96.7 -> 0.00 mm
- net /COL11: track 96.6 -> 0.00 mm
- net /COL12: track 95.5 -> 0.00 mm
- net /COL13: track 94.7 -> 0.00 mm
- net /COL0: track 90.4 -> 0.00 mm
- net /COL9: track 73.5 -> 0.00 mm
- net /COL5: track 73.5 -> 0.00 mm
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- added copper zone on F.Cu, net (none)
Other:
- board size 284.5 x 94 mm -> 480 x 154 mm
