File: tutorial.kicad_pcb (KiCad board)
At the start: 2 copper layers, 480 x 154 mm, 244 parts, among them SW0:0 ESC, SW0:1 1, SW0:10 0, SW0:11 -, SW0:12 =, SW0:13 BCKSPC, SW0:14 INS, SW0:15 HOME, SW0:2 2, SW0:3 3, SW0:4 4, SW0:5 5, SW0:6 6, SW0:7 7, SW0:8 8, SW0:9 9, SW1:0 PAGE_UP, SW1:1 TAB, SW1:10 O, SW1:11 P, SW1:12 [, SW1:13 ], SW1:14 \, SW1:15 DEL, SW1:2 Q, SW1:3 W, SW1:4 E, SW1:5 R, SW1:6 T, SW1:7 Y, SW1:8 U, SW1:9 I, SW2:0 END, SW2:1 PAGE_DOWN, SW2:10 K, SW2:11 L, SW2:12 ;, SW2:13 `, SW2:14 ENTER, SW2:15 LEFT, SW2:2 CAPSLOCK, SW2:3 A, SW2:4 S, SW2:5 D, SW2:6 F, SW2:7 G, SW2:8 H, SW2:9 J, SW3:0 RIGHT, SW3:1 L_SHIFT, SW3:10 ., SW3:11 /, SW3:12 R_SHIFT, SW3:13 UP, SW3:14 DOWN, SW3:15 L_CTRL, SW3:2 Z, SW3:3 X, SW3:4 C, SW3:5 V, SW3:6 B, SW3:7 N, SW3:8 M, SW3:9 ,, SW4:0 L_SUPER, SW4:1 L_ALT, SW4:10 KEYPAD_1, SW4:11 KEYPAD_2, SW4:12 KEYPAD_3, SW4:13 KEYPAD_4, SW4:14 KEYPAD_5, SW4:15 KEYPAD_6, SW4:2 SPACE, SW4:3 R_ALT, SW4:4 R_SUPER, SW4:5 MENU, SW4:6 R_CTRL, SW4:7 KEYPAD_0, SW4:8 KEYPAD_DEL, SW4:9 KEYPAD_ENTER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

Commit message: 3° commit
Parts:
- removed ? (x2): , Wire_Pads:SolderWirePad_single_2-5mmDrill
- removed the SW4:2 at (205.5, 230.0)
- moved SW4:2 0.27 mm to (205.7, 229.9)
Connections:
- SW0:0 pad 3: (no net) -> /LED_MATRIX_ANODE
- SW0:1 pad 3: (no net) -> /LED_MATRIX_ANODE
- SW0:10 pad 3: (no net) -> /LED_MATRIX_ANODE
- SW0:11 pad 3: (no net) -> /LED_MATRIX_ANODE
- SW0:12 pad 3: (no net) -> /LED_MATRIX_ANODE
- SW0:13 pad 3: (no net) -> /LED_MATRIX_ANODE
- SW0:14 pad 3: (no net) -> /LED_MATRIX_ANODE
- SW0:15 pad 3: (no net) -> /LED_MATRIX_ANODE
- SW0:2 pad 3: (no net) -> /LED_MATRIX_ANODE
- SW0:3 pad 3: (no net) -> /LED_MATRIX_ANODE
- SW0:4 pad 3: (no net) -> /LED_MATRIX_ANODE
- SW0:5 pad 3: (no net) -> /LED_MATRIX_ANODE
- SW0:6 pad 3: (no net) -> /LED_MATRIX_ANODE
- SW0:7 pad 3: (no net) -> /LED_MATRIX_ANODE
- SW0:8 pad 3: (no net) -> /LED_MATRIX_ANODE
- SW0:9 pad 3: (no net) -> /LED_MATRIX_ANODE
- SW1:0 pad 3: (no net) -> /LED_MATRIX_ANODE
- SW1:1 pad 3: (no net) -> /LED_MATRIX_ANODE
- SW1:10 pad 3: (no net) -> /LED_MATRIX_ANODE
- SW1:11 pad 3: (no net) -> /LED_MATRIX_ANODE
- SW1:12 pad 3: (no net) -> /LED_MATRIX_ANODE
- SW1:13 pad 3: (no net) -> /LED_MATRIX_ANODE
- SW1:14 pad 3: (no net) -> /LED_MATRIX_ANODE
- SW1:15 pad 3: (no net) -> /LED_MATRIX_ANODE
- SW1:2 pad 3: (no net) -> /LED_MATRIX_ANODE
- SW1:3 pad 3: (no net) -> /LED_MATRIX_ANODE
- SW1:4 pad 3: (no net) -> /LED_MATRIX_ANODE
- SW1:5 pad 3: (no net) -> /LED_MATRIX_ANODE
- SW1:6 pad 3: (no net) -> /LED_MATRIX_ANODE
- SW1:7 pad 3: (no net) -> /LED_MATRIX_ANODE
- SW1:8 pad 3: (no net) -> /LED_MATRIX_ANODE
- SW1:9 pad 3: (no net) -> /LED_MATRIX_ANODE
- SW2:0 pad 3: (no net) -> /LED_MATRIX_ANODE
- SW2:1 pad 3: (no net) -> /LED_MATRIX_ANODE
- SW2:10 pad 3: (no net) -> /LED_MATRIX_ANODE
- SW2:11 pad 3: (no net) -> /LED_MATRIX_ANODE
- SW2:12 pad 3: (no net) -> /LED_MATRIX_ANODE
- SW2:13 pad 3: (no net) -> /LED_MATRIX_ANODE
- SW2:14 pad 3: (no net) -> /LED_MATRIX_ANODE
- SW2:15 pad 3: (no net) -> /LED_MATRIX_ANODE
- SW2:2 pad 3: (no net) -> /LED_MATRIX_ANODE
- SW2:3 pad 3: (no net) -> /LED_MATRIX_ANODE
- SW2:4 pad 3: (no net) -> /LED_MATRIX_ANODE
- SW2:5 pad 3: (no net) -> /LED_MATRIX_ANODE
- SW2:6 pad 3: (no net) -> /LED_MATRIX_ANODE
- SW2:7 pad 3: (no net) -> /LED_MATRIX_ANODE
- SW2:8 pad 3: (no net) -> /LED_MATRIX_ANODE
- SW2:9 pad 3: (no net) -> /LED_MATRIX_ANODE
- SW3:0 pad 3: (no net) -> /LED_MATRIX_ANODE
- SW3:1 pad 3: (no net) -> /LED_MATRIX_ANODE
- SW3:10 pad 3: (no net) -> /LED_MATRIX_ANODE
- SW3:11 pad 3: (no net) -> /LED_MATRIX_ANODE
- SW3:12 pad 3: (no net) -> /LED_MATRIX_ANODE
- SW3:13 pad 3: (no net) -> /LED_MATRIX_ANODE
- SW3:14 pad 3: (no net) -> /LED_MATRIX_ANODE
- SW3:15 pad 3: (no net) -> /LED_MATRIX_ANODE
- SW3:2 pad 3: (no net) -> /LED_MATRIX_ANODE
- SW3:3 pad 3: (no net) -> /LED_MATRIX_ANODE
- SW3:4 pad 3: (no net) -> /LED_MATRIX_ANODE
- SW3:5 pad 3: (no net) -> /LED_MATRIX_ANODE
- SW3:6 pad 3: (no net) -> /LED_MATRIX_ANODE
- SW3:7 pad 3: (no net) -> /LED_MATRIX_ANODE
- SW3:8 pad 3: (no net) -> /LED_MATRIX_ANODE
- SW3:9 pad 3: (no net) -> /LED_MATRIX_ANODE
- SW4:0 pad 3: (no net) -> /LED_MATRIX_ANODE
- SW4:1 pad 3: (no net) -> /LED_MATRIX_ANODE
- SW4:10 pad 3: (no net) -> /LED_MATRIX_ANODE
- SW4:11 pad 3: (no net) -> /LED_MATRIX_ANODE
- SW4:12 pad 3: (no net) -> /LED_MATRIX_ANODE
- SW4:13 pad 3: (no net) -> /LED_MATRIX_ANODE
- SW4:14 pad 3: (no net) -> /LED_MATRIX_ANODE
- SW4:15 pad 3: (no net) -> /LED_MATRIX_ANODE
- SW4:2 pad 3: (no net) -> /LED_MATRIX_ANODE
- SW4:3 pad 3: (no net) -> /LED_MATRIX_ANODE
- SW4:4 pad 3: (no net) -> /LED_MATRIX_ANODE
- SW4:5 pad 3: (no net) -> /LED_MATRIX_ANODE
- SW4:6 pad 3: (no net) -> /LED_MATRIX_ANODE
- SW4:7 pad 3: (no net) -> /LED_MATRIX_ANODE
- SW4:8 pad 3: (no net) -> /LED_MATRIX_ANODE
- SW4:9 pad 3: (no net) -> /LED_MATRIX_ANODE
- SW5:0 pad 3: (no net) -> /LED_MATRIX_ANODE
- SW5:1 pad 3: (no net) -> /LED_MATRIX_ANODE
- SW5:10 pad 3: (no net) -> /LED_MATRIX_ANODE
- SW5:11 pad 3: (no net) -> /LED_MATRIX_ANODE
- SW5:12 pad 3: (no net) -> /LED_MATRIX_ANODE
- SW5:13 pad 3: (no net) -> /LED_MATRIX_ANODE
- SW5:14 pad 3: (no net) -> /LED_MATRIX_ANODE
- SW5:15 pad 3: (no net) -> /LED_MATRIX_ANODE
- SW5:2 pad 3: (no net) -> /LED_MATRIX_ANODE
- SW5:3 pad 3: (no net) -> /LED_MATRIX_ANODE
- SW5:4 pad 3: (no net) -> /LED_MATRIX_ANODE
- SW5:5 pad 3: (no net) -> /LED_MATRIX_ANODE
- SW5:6 pad 3: (no net) -> /LED_MATRIX_ANODE
- SW5:7 pad 3: (no net) -> /LED_MATRIX_ANODE
- SW5:8 pad 3: (no net) -> /LED_MATRIX_ANODE
- SW5:9 pad 3: (no net) -> /LED_MATRIX_ANODE
- SW6:0 pad 3: (no net) -> /LED_MATRIX_ANODE
- SW6:1 pad 3: (no net) -> /LED_MATRIX_ANODE
- SW6:10 pad 3: (no net) -> /LED_MATRIX_ANODE
- SW6:11 pad 3: (no net) -> /LED_MATRIX_ANODE
- SW6:12 pad 3: (no net) -> /LED_MATRIX_ANODE
- SW6:13 pad 3: (no net) -> /LED_MATRIX_ANODE
- SW6:14 pad 3: (no net) -> /LED_MATRIX_ANODE
- SW6:15 pad 3: (no net) -> /LED_MATRIX_ANODE
- SW6:2 pad 3: (no net) -> /LED_MATRIX_ANODE
- SW6:3 pad 3: (no net) -> /LED_MATRIX_ANODE
- SW6:4 pad 3: (no net) -> /LED_MATRIX_ANODE
- SW6:5 pad 3: (no net) -> /LED_MATRIX_ANODE
- SW6:6 pad 3: (no net) -> /LED_MATRIX_ANODE
- SW6:7 pad 3: (no net) -> /LED_MATRIX_ANODE
- SW6:8 pad 3: (no net) -> /LED_MATRIX_ANODE
- SW6:9 pad 3: (no net) -> /LED_MATRIX_ANODE
- SW7:0 pad 3: (no net) -> /LED_MATRIX_ANODE
- SW7:1 pad 3: (no net) -> /LED_MATRIX_ANODE
- SW7:2 pad 3: (no net) -> /LED_MATRIX_ANODE
- SW7:3 pad 3: (no net) -> /LED_MATRIX_ANODE
- SW7:4 pad 3: (no net) -> Net-(SW7:4-Pad3)
- SW7:5 pad 3: (no net) -> Net-(SW7:5-Pad3)
Routing:
- net /LED_MATRIX_KATODE: track 0.00 -> 3310.3 mm, vias 0 -> 27
- net /LED_MATRIX_ANODE: track 0.00 -> 3254.8 mm, vias 0 -> 35
- net /COL8: track 203.3 -> 874.2 mm, vias 1 -> 15
- net /COL6: track 136.8 -> 800.8 mm, vias 0 -> 6
- net /COL0: track 113.5 -> 736.9 mm, vias 0 -> 11
- net /COL10: track 181.0 -> 767.1 mm, vias 0 -> 9
- net /COL4: track 137.1 -> 705.2 mm, vias 0 -> 15
- net /COL3: track 183.7 -> 713.1 mm, vias 0 -> 10
- net /COL9: track 182.9 -> 646.4 mm, vias 0 -> 5
- net /COL15: track 480.9 -> 939.0 mm, vias 5 -> 17
- net /COL13: track 146.2 -> 568.2 mm, vias 0 -> 7
- net /COL1: track 119.1 -> 538.0 mm, vias 0 -> 8
- net /COL5: track 139.5 -> 498.2 mm, vias 0 -> 9
- net /COL11: track 182.6 -> 527.7 mm, vias 0 -> 10
- net /COL12: track 216.5 -> 520.8 mm, vias 0 -> 7
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
Commit message: another little step
Routing:
- net /COL10: track 767.1 -> 223.6 mm, vias 9 -> 2
- net /COL9: track 646.4 -> 159.3 mm, vias 5 -> 3
- net /COL12: track 520.8 -> 158.9 mm, vias 7 -> 3
- net /COL3: track 713.1 -> 367.1 mm, vias 10 -> 9
- net /COL6: track 800.8 -> 459.3 mm, vias 6 -> 14
- net /LED_MATRIX_KATODE: track 3310.3 -> 3034.8 mm, vias 27 -> 16
- net /LED_MATRIX_ANODE: track 3254.8 -> 2995.6 mm, vias 35 -> 15
- net /ROW5: track 450.1 -> 670.6 mm, vias 1 -> 4
- net /COL2: track 340.4 -> 504.6 mm, vias 5 -> 6
- net /ROW3: track 453.7 -> 612.4 mm, vias 1 -> 4
- net /COL15: track 939.0 -> 780.7 mm, vias 17 -> 7
- net /COL14: track 582.2 -> 429.0 mm, vias 5 -> 8
- net /COL7: track 435.6 -> 582.2 mm, vias 8 -> 10
- net /COL11: track 527.7 -> 657.8 mm, vias 10 -> 12
- net /COL5: track 498.2 -> 624.3 mm, vias 9 -> 18
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
Commit message: sbroglio terminato
Parts:
- moved L2 79.8 mm to (415.9, 86.4)
- moved L3 78.9 mm to (432.4, 86.4)
- moved L1 78.0 mm to (399.4, 87.0)
- moved R3 75.7 mm to (434.3, 99.7)
- moved R2 74.4 mm to (419.7, 99.7)
- moved R1 73.1 mm to (402.6, 99.7)
Routing:
- net /COL12: track 158.9 -> 853.8 mm, vias 3 -> 29
- net /COL9: track 159.3 -> 835.9 mm, vias 3 -> 16
- net /COL10: track 223.6 -> 843.9 mm, vias 2 -> 24
- net /COL3: track 367.1 -> 747.3 mm, vias 9 -> 13
- net /COL14: track 429.0 -> 684.3 mm, vias 8 -> 11
- net /COL6: track 459.3 -> 675.5 mm, vias 14 -> 19
- net /COL2: track 504.6 -> 707.5 mm, vias 6 -> 13
- net /LED_B: track 37.5 -> 224.8 mm, vias 0 -> 12
- net /COL1: track 661.7 -> 827.9 mm, vias 19 -> 29
- net /LED_C: track 32.4 -> 171.0 mm, vias 1 -> 2
- net /LED_A: track 53.2 -> 190.4 mm, vias 1 -> 3
- net /ROW7: track 191.2 -> 322.4 mm, vias 0 -> 7
- net /COL7: track 582.2 -> 689.8 mm, vias 10 -> 12
- net /COL0: track 781.2 -> 873.7 mm, vias 15 -> 20
- net /COL5: track 624.3 -> 708.9 mm, vias 18 -> 16
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
Commit message: 4o step
Parts:
- added REF**: , Mounting_Holes:MountingHole_2.7mm_M2.5, F.Cu at (59.4, 141.0)
- added REF**: , Mounting_Holes:MountingHole_2.7mm_M2.5, F.Cu at (471.1, 168.4)
- moved SW5:7 63.9 mm to (471.2, 154.0)
- moved SW5:0 63.3 mm to (471.2, 182.8)
- moved SW4:9 62.8 mm to (471.2, 221.2)
- moved SW5:6 61.3 mm to (451.9, 154.0)
- moved SW5:3 60.8 mm to (451.9, 173.2)
- moved SW4:15 60.4 mm to (451.9, 192.4)
- moved SW4:12 60.1 mm to (452.0, 211.6)
- moved SW4:8 60.0 mm to (452.0, 230.8)
- moved D4:8 58.6 mm to (443.4, 231.2)
- moved SW5:5 58.5 mm to (432.7, 154.0)
- moved SW5:2 58.0 mm to (432.7, 173.2)
- moved SW4:14 57.7 mm to (432.7, 192.4)
- moved SW4:11 57.4 mm to (432.7, 211.6)
- moved D5:7 56.4 mm to (471.3, 162.6), turned to 0 degrees
- moved SW4:7 55.8 mm to (423.2, 230.8)
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Connections:
- SW0:0 pad 3: /LED_MATRIX_ANODE -> Net-(SW0:0-Pad3)
- SW0:0 pad 4: /LED_MATRIX_KATODE -> Net-(SW0:0-Pad4)
- SW0:1 pad 3: /LED_MATRIX_ANODE -> Net-(SW0:1-Pad3)
- SW0:1 pad 4: /LED_MATRIX_KATODE -> Net-(SW0:1-Pad4)
- SW0:10 pad 3: /LED_MATRIX_ANODE -> Net-(SW0:10-Pad3)
- SW0:10 pad 4: /LED_MATRIX_KATODE -> Net-(SW0:10-Pad4)
- SW0:11 pad 3: /LED_MATRIX_ANODE -> Net-(SW0:11-Pad3)
- SW0:11 pad 4: /LED_MATRIX_KATODE -> Net-(SW0:11-Pad4)
- SW0:12 pad 3: /LED_MATRIX_ANODE -> Net-(SW0:12-Pad3)
- SW0:12 pad 4: /LED_MATRIX_KATODE -> Net-(SW0:12-Pad4)
- SW0:13 pad 3: /LED_MATRIX_ANODE -> Net-(SW0:13-Pad3)
- SW0:13 pad 4: /LED_MATRIX_KATODE -> Net-(SW0:13-Pad4)
- SW0:14 pad 3: /LED_MATRIX_ANODE -> Net-(SW0:14-Pad3)
- SW0:14 pad 4: /LED_MATRIX_KATODE -> Net-(SW0:14-Pad4)
- SW0:15 pad 3: /LED_MATRIX_ANODE -> Net-(SW0:15-Pad3)
- SW0:15 pad 4: /LED_MATRIX_KATODE -> Net-(SW0:15-Pad4)
- SW0:2 pad 3: /LED_MATRIX_ANODE -> Net-(SW0:2-Pad3)
- SW0:2 pad 4: /LED_MATRIX_KATODE -> Net-(SW0:2-Pad4)
- SW0:3 pad 3: /LED_MATRIX_ANODE -> Net-(SW0:3-Pad3)
- SW0:3 pad 4: /LED_MATRIX_KATODE -> Net-(SW0:3-Pad4)
- SW0:4 pad 3: /LED_MATRIX_ANODE -> Net-(SW0:4-Pad3)
- SW0:4 pad 4: /LED_MATRIX_KATODE -> Net-(SW0:4-Pad4)
- SW0:5 pad 3: /LED_MATRIX_ANODE -> Net-(SW0:5-Pad3)
- SW0:5 pad 4: /LED_MATRIX_KATODE -> Net-(SW0:5-Pad4)
- SW0:6 pad 3: /LED_MATRIX_ANODE -> Net-(SW0:6-Pad3)
- SW0:6 pad 4: /LED_MATRIX_KATODE -> Net-(SW0:6-Pad4)
- SW0:7 pad 3: /LED_MATRIX_ANODE -> Net-(SW0:7-Pad3)
- SW0:7 pad 4: /LED_MATRIX_KATODE -> Net-(SW0:7-Pad4)
- SW0:8 pad 3: /LED_MATRIX_ANODE -> Net-(SW0:8-Pad3)
- SW0:8 pad 4: /LED_MATRIX_KATODE -> Net-(SW0:8-Pad4)
- SW0:9 pad 3: /LED_MATRIX_ANODE -> Net-(SW0:9-Pad3)
- SW0:9 pad 4: /LED_MATRIX_KATODE -> Net-(SW0:9-Pad4)
- SW1:0 pad 3: /LED_MATRIX_ANODE -> Net-(SW1:0-Pad3)
- SW1:0 pad 4: /LED_MATRIX_KATODE -> Net-(SW1:0-Pad4)
- SW1:1 pad 3: /LED_MATRIX_ANODE -> Net-(SW1:1-Pad3)
- SW1:1 pad 4: /LED_MATRIX_KATODE -> Net-(SW1:1-Pad4)
- SW1:10 pad 3: /LED_MATRIX_ANODE -> Net-(SW1:10-Pad3)
- SW1:10 pad 4: /LED_MATRIX_KATODE -> Net-(SW1:10-Pad4)
- SW1:11 pad 3: /LED_MATRIX_ANODE -> Net-(SW1:11-Pad3)
- SW1:11 pad 4: /LED_MATRIX_KATODE -> Net-(SW1:11-Pad4)
- SW1:12 pad 3: /LED_MATRIX_ANODE -> Net-(SW1:12-Pad3)
- SW1:12 pad 4: /LED_MATRIX_KATODE -> Net-(SW1:12-Pad4)
- SW1:13 pad 3: /LED_MATRIX_ANODE -> Net-(SW1:13-Pad3)
- SW1:13 pad 4: /LED_MATRIX_KATODE -> Net-(SW1:13-Pad4)
- SW1:14 pad 3: /LED_MATRIX_ANODE -> Net-(SW1:14-Pad3)
- SW1:14 pad 4: /LED_MATRIX_KATODE -> Net-(SW1:14-Pad4)
- SW1:15 pad 3: /LED_MATRIX_ANODE -> Net-(SW1:15-Pad3)
- SW1:15 pad 4: /LED_MATRIX_KATODE -> Net-(SW1:15-Pad4)
- SW1:2 pad 3: /LED_MATRIX_ANODE -> Net-(SW1:2-Pad3)
- SW1:2 pad 4: /LED_MATRIX_KATODE -> Net-(SW1:2-Pad4)
- SW1:3 pad 3: /LED_MATRIX_ANODE -> Net-(SW1:3-Pad3)
- SW1:3 pad 4: /LED_MATRIX_KATODE -> Net-(SW1:3-Pad4)
- SW1:4 pad 3: /LED_MATRIX_ANODE -> Net-(SW1:4-Pad3)
- SW1:4 pad 4: /LED_MATRIX_KATODE -> Net-(SW1:4-Pad4)
- SW1:5 pad 3: /LED_MATRIX_ANODE -> Net-(SW1:5-Pad3)
- SW1:5 pad 4: /LED_MATRIX_KATODE -> Net-(SW1:5-Pad4)
- SW1:6 pad 3: /LED_MATRIX_ANODE -> Net-(SW1:6-Pad3)
- SW1:6 pad 4: /LED_MATRIX_KATODE -> Net-(SW1:6-Pad4)
- SW1:7 pad 3: /LED_MATRIX_ANODE -> Net-(SW1:7-Pad3)
- SW1:7 pad 4: /LED_MATRIX_KATODE -> Net-(SW1:7-Pad4)
- SW1:8 pad 3: /LED_MATRIX_ANODE -> Net-(SW1:8-Pad3)
- SW1:8 pad 4: /LED_MATRIX_KATODE -> Net-(SW1:8-Pad4)
- SW1:9 pad 3: /LED_MATRIX_ANODE -> Net-(SW1:9-Pad3)
- SW1:9 pad 4: /LED_MATRIX_KATODE -> Net-(SW1:9-Pad4)
- SW2:0 pad 3: /LED_MATRIX_ANODE -> Net-(SW2:0-Pad3)
- SW2:0 pad 4: /LED_MATRIX_KATODE -> Net-(SW2:0-Pad4)
- SW2:1 pad 3: /LED_MATRIX_ANODE -> Net-(SW2:1-Pad3)
- SW2:1 pad 4: /LED_MATRIX_KATODE -> Net-(SW2:1-Pad4)
- SW2:10 pad 3: /LED_MATRIX_ANODE -> Net-(SW2:10-Pad3)
- SW2:10 pad 4: /LED_MATRIX_KATODE -> Net-(SW2:10-Pad4)
- SW2:11 pad 3: /LED_MATRIX_ANODE -> Net-(SW2:11-Pad3)
- SW2:11 pad 4: /LED_MATRIX_KATODE -> Net-(SW2:11-Pad4)
- SW2:12 pad 3: /LED_MATRIX_ANODE -> Net-(SW2:12-Pad3)
- SW2:12 pad 4: /LED_MATRIX_KATODE -> Net-(SW2:12-Pad4)
- SW2:13 pad 3: /LED_MATRIX_ANODE -> Net-(SW2:13-Pad3)
- SW2:13 pad 4: /LED_MATRIX_KATODE -> Net-(SW2:13-Pad4)
- SW2:14 pad 3: /LED_MATRIX_ANODE -> Net-(SW2:14-Pad3)
- SW2:14 pad 4: /LED_MATRIX_KATODE -> Net-(SW2:14-Pad4)
- SW2:15 pad 3: /LED_MATRIX_ANODE -> Net-(SW2:15-Pad3)
- SW2:15 pad 4: /LED_MATRIX_KATODE -> Net-(SW2:15-Pad4)
- SW2:2 pad 3: /LED_MATRIX_ANODE -> Net-(SW2:2-Pad3)
- SW2:2 pad 4: /LED_MATRIX_KATODE -> Net-(SW2:2-Pad4)
- SW2:3 pad 3: /LED_MATRIX_ANODE -> Net-(SW2:3-Pad3)
- SW2:3 pad 4: /LED_MATRIX_KATODE -> Net-(SW2:3-Pad4)
- SW2:4 pad 3: /LED_MATRIX_ANODE -> Net-(SW2:4-Pad3)
- SW2:4 pad 4: /LED_MATRIX_KATODE -> Net-(SW2:4-Pad4)
- SW2:5 pad 3: /LED_MATRIX_ANODE -> Net-(SW2:5-Pad3)
- SW2:5 pad 4: /LED_MATRIX_KATODE -> Net-(SW2:5-Pad4)
- SW2:6 pad 3: /LED_MATRIX_ANODE -> Net-(SW2:6-Pad3)
- SW2:6 pad 4: /LED_MATRIX_KATODE -> Net-(SW2:6-Pad4)
- SW2:7 pad 3: /LED_MATRIX_ANODE -> Net-(SW2:7-Pad3)
- SW2:7 pad 4: /LED_MATRIX_KATODE -> Net-(SW2:7-Pad4)
- SW2:8 pad 3: /LED_MATRIX_ANODE -> Net-(SW2:8-Pad3)
- SW2:8 pad 4: /LED_MATRIX_KATODE -> Net-(SW2:8-Pad4)
- SW2:9 pad 3: /LED_MATRIX_ANODE -> Net-(SW2:9-Pad3)
- SW2:9 pad 4: /LED_MATRIX_KATODE -> Net-(SW2:9-Pad4)
- SW3:0 pad 3: /LED_MATRIX_ANODE -> Net-(SW3:0-Pad3)
- SW3:0 pad 4: /LED_MATRIX_KATODE -> Net-(SW3:0-Pad4)
- SW3:1 pad 3: /LED_MATRIX_ANODE -> Net-(SW3:1-Pad3)
- SW3:1 pad 4: /LED_MATRIX_KATODE -> Net-(SW3:1-Pad4)
- SW3:10 pad 3: /LED_MATRIX_ANODE -> Net-(SW3:10-Pad3)
- SW3:10 pad 4: /LED_MATRIX_KATODE -> Net-(SW3:10-Pad4)
- SW3:11 pad 3: /LED_MATRIX_ANODE -> Net-(SW3:11-Pad3)
- SW3:11 pad 4: /LED_MATRIX_KATODE -> Net-(SW3:11-Pad4)
- SW3:12 pad 3: /LED_MATRIX_ANODE -> Net-(SW3:12-Pad3)
- SW3:12 pad 4: /LED_MATRIX_KATODE -> Net-(SW3:12-Pad4)
- SW3:13 pad 3: /LED_MATRIX_ANODE -> Net-(SW3:13-Pad3)
- SW3:13 pad 4: /LED_MATRIX_KATODE -> Net-(SW3:13-Pad4)
- SW3:14 pad 3: /LED_MATRIX_ANODE -> Net-(SW3:14-Pad3)
- SW3:14 pad 4: /LED_MATRIX_KATODE -> Net-(SW3:14-Pad4)
- SW3:15 pad 3: /LED_MATRIX_ANODE -> Net-(SW3:15-Pad3)
- SW3:15 pad 4: /LED_MATRIX_KATODE -> Net-(SW3:15-Pad4)
- SW3:2 pad 3: /LED_MATRIX_ANODE -> Net-(SW3:2-Pad3)
- SW3:2 pad 4: /LED_MATRIX_KATODE -> Net-(SW3:2-Pad4)
- SW3:3 pad 3: /LED_MATRIX_ANODE -> Net-(SW3:3-Pad3)
- SW3:3 pad 4: /LED_MATRIX_KATODE -> Net-(SW3:3-Pad4)
- SW3:4 pad 3: /LED_MATRIX_ANODE -> Net-(SW3:4-Pad3)
- SW3:4 pad 4: /LED_MATRIX_KATODE -> Net-(SW3:4-Pad4)
- SW3:5 pad 3: /LED_MATRIX_ANODE -> Net-(SW3:5-Pad3)
- SW3:5 pad 4: /LED_MATRIX_KATODE -> Net-(SW3:5-Pad4)
- SW3:6 pad 3: /LED_MATRIX_ANODE -> Net-(SW3:6-Pad3)
- SW3:6 pad 4: /LED_MATRIX_KATODE -> Net-(SW3:6-Pad4)
- SW3:7 pad 3: /LED_MATRIX_ANODE -> Net-(SW3:7-Pad3)
- SW3:7 pad 4: /LED_MATRIX_KATODE -> Net-(SW3:7-Pad4)
- SW3:8 pad 3: /LED_MATRIX_ANODE -> Net-(SW3:8-Pad3)
- SW3:8 pad 4: /LED_MATRIX_KATODE -> Net-(SW3:8-Pad4)
- SW3:9 pad 3: /LED_MATRIX_ANODE -> Net-(SW3:9-Pad3)
- SW3:9 pad 4: /LED_MATRIX_KATODE -> Net-(SW3:9-Pad4)
- SW4:0 pad 3: /LED_MATRIX_ANODE -> Net-(SW4:0-Pad3)
- SW4:0 pad 4: /LED_MATRIX_KATODE -> Net-(SW4:0-Pad4)
- SW4:1 pad 3: /LED_MATRIX_ANODE -> Net-(SW4:1-Pad3)
- SW4:1 pad 4: /LED_MATRIX_KATODE -> Net-(SW4:1-Pad4)
- SW4:10 pad 3: /LED_MATRIX_ANODE -> Net-(SW4:10-Pad3)
- SW4:10 pad 4: /LED_MATRIX_KATODE -> Net-(SW4:10-Pad4)
- SW4:11 pad 3: /LED_MATRIX_ANODE -> Net-(SW4:11-Pad3)
- SW4:11 pad 4: /LED_MATRIX_KATODE -> Net-(SW4:11-Pad4)
- SW4:12 pad 3: /LED_MATRIX_ANODE -> Net-(SW4:12-Pad3)
- SW4:12 pad 4: /LED_MATRIX_KATODE -> Net-(SW4:12-Pad4)
- SW4:13 pad 3: /LED_MATRIX_ANODE -> Net-(SW4:13-Pad3)
- SW4:13 pad 4: /LED_MATRIX_KATODE -> Net-(SW4:13-Pad4)
- SW4:14 pad 3: /LED_MATRIX_ANODE -> Net-(SW4:14-Pad3)
- SW4:14 pad 4: /LED_MATRIX_KATODE -> Net-(SW4:14-Pad4)
- SW4:15 pad 3: /LED_MATRIX_ANODE -> Net-(SW4:15-Pad3)
- SW4:15 pad 4: /LED_MATRIX_KATODE -> Net-(SW4:15-Pad4)
- SW4:2 pad 3: /LED_MATRIX_ANODE -> Net-(SW4:2-Pad3)
- SW4:2 pad 4: /LED_MATRIX_KATODE -> Net-(SW4:2-Pad4)
- SW4:3 pad 3: /LED_MATRIX_ANODE -> Net-(SW4:3-Pad3)
- SW4:3 pad 4: /LED_MATRIX_KATODE -> Net-(SW4:3-Pad4)
- SW4:4 pad 3: /LED_MATRIX_ANODE -> Net-(SW4:4-Pad3)
- SW4:4 pad 4: /LED_MATRIX_KATODE -> Net-(SW4:4-Pad4)
- SW4:5 pad 3: /LED_MATRIX_ANODE -> Net-(SW4:5-Pad3)
- SW4:5 pad 4: /LED_MATRIX_KATODE -> Net-(SW4:5-Pad4)
- SW4:6 pad 3: /LED_MATRIX_ANODE -> Net-(SW4:6-Pad3)
- SW4:6 pad 4: /LED_MATRIX_KATODE -> Net-(SW4:6-Pad4)
- SW4:7 pad 3: /LED_MATRIX_ANODE -> Net-(SW4:7-Pad3)
- SW4:7 pad 4: /LED_MATRIX_KATODE -> Net-(SW4:7-Pad4)
- SW4:8 pad 3: /LED_MATRIX_ANODE -> Net-(SW4:8-Pad3)
- SW4:8 pad 4: /LED_MATRIX_KATODE -> Net-(SW4:8-Pad4)
- SW4:9 pad 3: /LED_MATRIX_ANODE -> Net-(SW4:9-Pad3)
- SW4:9 pad 4: /LED_MATRIX_KATODE -> Net-(SW4:9-Pad4)
- SW5:0 pad 3: /LED_MATRIX_ANODE -> Net-(SW5:0-Pad3)
- SW5:0 pad 4: /LED_MATRIX_KATODE -> Net-(SW5:0-Pad4)
- SW5:1 pad 3: /LED_MATRIX_ANODE -> Net-(SW5:1-Pad3)
- SW5:1 pad 4: /LED_MATRIX_KATODE -> Net-(SW5:1-Pad4)
- SW5:10 pad 3: /LED_MATRIX_ANODE -> Net-(SW5:10-Pad3)
- SW5:10 pad 4: /LED_MATRIX_KATODE -> Net-(SW5:10-Pad4)
- SW5:11 pad 3: /LED_MATRIX_ANODE -> Net-(SW5:11-Pad3)
- SW5:11 pad 4: /LED_MATRIX_KATODE -> Net-(SW5:11-Pad4)
- SW5:12 pad 3: /LED_MATRIX_ANODE -> Net-(SW5:12-Pad3)
- SW5:12 pad 4: /LED_MATRIX_KATODE -> Net-(SW5:12-Pad4)
- SW5:13 pad 3: /LED_MATRIX_ANODE -> Net-(SW5:13-Pad3)
- SW5:13 pad 4: /LED_MATRIX_KATODE -> Net-(SW5:13-Pad4)
- SW5:14 pad 3: /LED_MATRIX_ANODE -> Net-(SW5:14-Pad3)
- SW5:14 pad 4: /LED_MATRIX_KATODE -> Net-(SW5:14-Pad4)
- SW5:15 pad 3: /LED_MATRIX_ANODE -> Net-(SW5:15-Pad3)
- SW5:15 pad 4: /LED_MATRIX_KATODE -> Net-(SW5:15-Pad4)
- SW5:2 pad 3: /LED_MATRIX_ANODE -> Net-(SW5:2-Pad3)
- SW5:2 pad 4: /LED_MATRIX_KATODE -> Net-(SW5:2-Pad4)
- SW5:3 pad 3: /LED_MATRIX_ANODE -> Net-(SW5:3-Pad3)
- SW5:3 pad 4: /LED_MATRIX_KATODE -> Net-(SW5:3-Pad4)
- SW5:4 pad 3: /LED_MATRIX_ANODE -> Net-(SW5:4-Pad3)
- SW5:4 pad 4: /LED_MATRIX_KATODE -> Net-(SW5:4-Pad4)
- SW5:5 pad 3: /LED_MATRIX_ANODE -> Net-(SW5:5-Pad3)
- SW5:5 pad 4: /LED_MATRIX_KATODE -> Net-(SW5:5-Pad4)
- SW5:6 pad 3: /LED_MATRIX_ANODE -> Net-(SW5:6-Pad3)
- SW5:6 pad 4: /LED_MATRIX_KATODE -> Net-(SW5:6-Pad4)
- SW5:7 pad 3: /LED_MATRIX_ANODE -> Net-(SW5:7-Pad3)
- SW5:7 pad 4: /LED_MATRIX_KATODE -> Net-(SW5:7-Pad4)
- SW5:8 pad 3: /LED_MATRIX_ANODE -> Net-(SW5:8-Pad3)
- SW5:8 pad 4: /LED_MATRIX_KATODE -> Net-(SW5:8-Pad4)
- SW5:9 pad 3: /LED_MATRIX_ANODE -> Net-(SW5:9-Pad3)
- SW5:9 pad 4: /LED_MATRIX_KATODE -> Net-(SW5:9-Pad4)
- SW6:0 pad 3: /LED_MATRIX_ANODE -> Net-(SW6:0-Pad3)
- SW6:0 pad 4: /LED_MATRIX_KATODE -> Net-(SW6:0-Pad4)
- SW6:1 pad 3: /LED_MATRIX_ANODE -> Net-(SW6:1-Pad3)
- SW6:1 pad 4: /LED_MATRIX_KATODE -> Net-(SW6:1-Pad4)
- SW6:10 pad 3: /LED_MATRIX_ANODE -> Net-(SW6:10-Pad3)
- SW6:10 pad 4: /LED_MATRIX_KATODE -> Net-(SW6:10-Pad4)
- SW6:11 pad 3: /LED_MATRIX_ANODE -> Net-(SW6:11-Pad3)
- SW6:11 pad 4: /LED_MATRIX_KATODE -> Net-(SW6:11-Pad4)
- SW6:12 pad 3: /LED_MATRIX_ANODE -> Net-(SW6:12-Pad3)
- SW6:12 pad 4: /LED_MATRIX_KATODE -> Net-(SW6:12-Pad4)
- SW6:13 pad 3: /LED_MATRIX_ANODE -> Net-(SW6:13-Pad3)
- SW6:13 pad 4: /LED_MATRIX_KATODE -> Net-(SW6:13-Pad4)
- SW6:14 pad 3: /LED_MATRIX_ANODE -> Net-(SW6:14-Pad3)
- SW6:14 pad 4: /LED_MATRIX_KATODE -> Net-(SW6:14-Pad4)
- SW6:15 pad 3: /LED_MATRIX_ANODE -> Net-(SW6:15-Pad3)
- SW6:15 pad 4: /LED_MATRIX_KATODE -> Net-(SW6:15-Pad4)
- SW6:2 pad 3: /LED_MATRIX_ANODE -> Net-(SW6:2-Pad3)
- SW6:2 pad 4: /LED_MATRIX_KATODE -> Net-(SW6:2-Pad4)
- SW6:3 pad 3: /LED_MATRIX_ANODE -> Net-(SW6:3-Pad3)
- SW6:3 pad 4: /LED_MATRIX_KATODE -> Net-(SW6:3-Pad4)
- SW6:4 pad 3: /LED_MATRIX_ANODE -> Net-(SW6:4-Pad3)
- SW6:4 pad 4: /LED_MATRIX_KATODE -> Net-(SW6:4-Pad4)
- SW6:5 pad 3: /LED_MATRIX_ANODE -> Net-(SW6:5-Pad3)
- SW6:5 pad 4: /LED_MATRIX_KATODE -> Net-(SW6:5-Pad4)
- SW6:6 pad 3: /LED_MATRIX_ANODE -> Net-(SW6:6-Pad3)
- SW6:6 pad 4: /LED_MATRIX_KATODE -> Net-(SW6:6-Pad4)
- SW6:7 pad 3: /LED_MATRIX_ANODE -> Net-(SW6:7-Pad3)
- SW6:7 pad 4: /LED_MATRIX_KATODE -> Net-(SW6:7-Pad4)
- SW6:8 pad 3: /LED_MATRIX_ANODE -> Net-(SW6:8-Pad3)
- SW6:8 pad 4: /LED_MATRIX_KATODE -> Net-(SW6:8-Pad4)
- SW6:9 pad 3: /LED_MATRIX_ANODE -> Net-(SW6:9-Pad3)
- SW6:9 pad 4: /LED_MATRIX_KATODE -> Net-(SW6:9-Pad4)
- SW7:0 pad 3: /LED_MATRIX_ANODE -> Net-(SW7:0-Pad3)
- SW7:0 pad 4: /LED_MATRIX_KATODE -> Net-(SW7:0-Pad4)
- SW7:1 pad 3: /LED_MATRIX_ANODE -> Net-(SW7:1-Pad3)
- SW7:1 pad 4: /LED_MATRIX_KATODE -> Net-(SW7:1-Pad4)
- SW7:2 pad 3: /LED_MATRIX_ANODE -> Net-(SW7:2-Pad3)
- SW7:2 pad 4: /LED_MATRIX_KATODE -> Net-(SW7:2-Pad4)
- SW7:3 pad 3: /LED_MATRIX_ANODE -> Net-(SW7:3-Pad3)
- SW7:3 pad 4: /LED_MATRIX_KATODE -> Net-(SW7:3-Pad4)
Routing:
- net /LED_MATRIX_KATODE: track 3034.4 -> 0.00 mm, vias 16 -> 0
- net /LED_MATRIX_ANODE: track 3004.9 -> 0.00 mm, vias 18 -> 0
- net /COL0: track 873.7 -> 125.9 mm, vias 20 -> 2
- net /COL9: track 835.9 -> 123.3 mm, vias 16 -> 3
- net /COL4: track 723.1 -> 93.7 mm, vias 10 -> 2
- net /COL1: track 827.9 -> 237.7 mm, vias 29 -> 6
- net /COL12: track 853.8 -> 290.2 mm, vias 29 -> 5
- net /COL3: track 747.3 -> 187.3 mm, vias 13 -> 6
- net /COL7: track 689.8 -> 139.5 mm, vias 12 -> 2
- net /COL5: track 708.9 -> 176.3 mm, vias 16 -> 7
- net /COL15: track 841.6 -> 346.9 mm, vias 13 -> 8
- net /COL14: track 684.3 -> 223.2 mm
- net /COL2: track 707.5 -> 260.2 mm, vias 13 -> 6
- net /COL10: track 843.9 -> 421.1 mm, vias 24 -> 11
- net /COL8: track 799.2 -> 424.6 mm, vias 15 -> 8
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- removed copper zone on F.Cu, net (none)
Other:
- board outline removed
