File: scdm_kicad_3_pcb.kicad_pcb (KiCad board)
At the start: 2 copper layers, 243 parts, among them SW0:0 ESC, SW0:1 1, SW0:10 0, SW0:11 -, SW0:12 =, SW0:13 BCKSPC, SW0:14 INS, SW0:15 HOME, SW0:2 2, SW0:3 3, SW0:4 4, SW0:5 5, SW0:6 6, SW0:7 7, SW0:8 8, SW0:9 9, SW1:0 PAGE_UP, SW1:1 TAB, SW1:10 O, SW1:11 P, SW1:12 [, SW1:13 ], SW1:14 \, SW1:15 DEL, SW1:2 Q, SW1:3 W, SW1:4 E, SW1:5 R, SW1:6 T, SW1:7 Y, SW1:8 U, SW1:9 I, SW2:0 END, SW2:1 PAGE_DOWN, SW2:10 K, SW2:11 L, SW2:12 ;, SW2:13 `, SW2:14 ENTER, SW2:15 LEFT, SW2:2 CAPSLOCK, SW2:3 A, SW2:4 S, SW2:5 D, SW2:6 F, SW2:7 G, SW2:8 H, SW2:9 J, SW3:0 RIGHT, SW3:1 L_SHIFT, SW3:10 ., SW3:11 /, SW3:12 R_SHIFT, SW3:13 UP, SW3:14 DOWN, SW3:15 L_CTRL, SW3:2 Z, SW3:3 X, SW3:4 C, SW3:5 V, SW3:6 B, SW3:7 N, SW3:8 M, SW3:9 ,, SW4:0 L_SUPER, SW4:1 L_ALT, SW4:10 KEYPAD_1, SW4:11 KEYPAD_2, SW4:12 KEYPAD_3, SW4:13 KEYPAD_4, SW4:14 KEYPAD_5, SW4:15 KEYPAD_6, SW4:2 SPACE, SW4:3 R_ALT, SW4:4 R_SUPER, SW4:5 MENU, SW4:6 R_CTRL, SW4:7 KEYPAD_0, SW4:8 KEYPAD_DEL, SW4:9 KEYPAD_ENTER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

Commit message: 4o step
Parts:
- moved D5:8 17.2 mm to (60.0, 145.4)
- moved D4:1 17.1 mm to (102.3, 231.3), turned to 90 degrees
- moved U1 14.1 mm to (432.4, 122.7)
- moved D6:9 12.2 mm to (98.0, 109.0), turned to 270 degrees
- moved D4:9 12.0 mm to (462.6, 221.7), turned to 90 degrees
- moved D0:1 12.0 mm to (69.9, 154.5), turned to 270 degrees
- moved D7:2 12.0 mm to (295.2, 109.2), turned to 270 degrees
- moved D1:14 12.0 mm to (309.5, 173.7), turned to 270 degrees
- moved D5:1 12.0 mm to (404.9, 173.7), turned to 90 degrees
- moved D5:3 12.0 mm to (443.3, 173.7), turned to 90 degrees
- moved D7:3 12.0 mm to (314.4, 109.3), turned to 270 degrees
- moved D0:12 12.0 mm to (281.3, 154.5), turned to 270 degrees
- moved D0:13 12.0 mm to (307.5, 154.5), turned to 270 degrees
- moved D0:7 12.0 mm to (185.1, 154.5), turned to 270 degrees
- moved D0:8 12.0 mm to (204.5, 154.5), turned to 270 degrees
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Routing:
- net /COL6: track 93.7 -> 263.2 mm, vias 2 -> 7
- net /ROW4: track 456.5 -> 602.1 mm, vias 2 -> 1
- net /COL15: track 235.9 -> 97.9 mm, vias 8 -> 1
- net /COL7: track 139.5 -> 277.0 mm, vias 2 -> 10
- net /COL1: track 237.7 -> 113.5 mm, vias 6 -> 2
- net /ROW7: track 184.2 -> 61.0 mm, vias 1 -> 0
- net /LED_A: track 0.11 -> 120.9 mm, vias 0 -> 1
- net /LED_B: track 0.11 -> 104.6 mm, vias 0 -> 2
- net /LED_C: track 0.11 -> 85.5 mm, vias 0 -> 2
- net /COL14: track 91.0 -> 173.3 mm, vias 2 -> 5
- net /ROW2: track 332.9 -> 280.8 mm, vias 2 -> 0
- net /COL3: track 187.3 -> 148.1 mm, vias 6 -> 8
- net /COL11: track 246.3 -> 208.0 mm, vias 5 -> 7
- net /COL12: track 290.2 -> 253.5 mm, vias 5 -> 3
- net GND: track 0.93 -> 36.4 mm
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Other:
- copper layers 2 -> 4
