File: tutorial.sch (KiCad schematic (older format))
At the start: 239 parts, among them SW0:0 ESC, SW0:1 1, SW0:10 0, SW0:11 -, SW0:12 =, SW0:13 BCKSPC, SW0:14 INS, SW0:15 HOME, SW0:2 2, SW0:3 3, SW0:4 4, SW0:5 5, SW0:6 6, SW0:7 7, SW0:8 8, SW0:9 9, SW1:0 PAGE_UP, SW1:1 TAB, SW1:10 O, SW1:11 P, SW1:12 [, SW1:13 ], SW1:14 \\, SW1:15 DEL, SW1:2 Q, SW1:3 W, SW1:4 E, SW1:5 R, SW1:6 T, SW1:7 Y, SW1:8 U, SW1:9 I, SW2:0 END, SW2:1 PAGE_DOWN, SW2:10 K, SW2:11 L, SW2:12 ;, SW2:13 `, SW2:14 ENTER, SW2:15 LEFT, SW2:2 CAPSLOCK, SW2:3 A, SW2:4 S, SW2:5 D, SW2:6 F, SW2:7 G, SW2:8 H, SW2:9 J, SW3:0 RIGHT, SW3:1 L_SHIFT, SW3:10 ., SW3:11 /, SW3:12 R_SHIFT, SW3:13 UP, SW3:14 DOWN, SW3:15 L_CTRL, SW3:2 Z, SW3:3 X, SW3:4 C, SW3:5 V, SW3:6 B, SW3:7 N, SW3:8 M, SW3:9 ,, SW4:0 L_SUPER, SW4:1 L_ALT, SW4:10 KEYPAD_1, SW4:11 KEYPAD_2, SW4:12 KEYPAD_3, SW4:13 KEYPAD_4, SW4:14 KEYPAD_5, SW4:15 KEYPAD_6, SW4:2 SPACE, SW4:3 R_ALT, SW4:4 R_SUPER, SW4:5 MENU, SW4:6 R_CTRL, SW4:7 KEYPAD_0, SW4:8 KEYPAD_DEL, SW4:9 KEYPAD_ENTER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

Commit message: second commit
Parts:
- added SW7:4: Fake1, Keyboard:CHERRY_PCB_100H_With_led2, symbol SWITCH_PUSH
- added SW7:5: Fake2, Keyboard:CHERRY_PCB_100H_With_led2, symbol SWITCH_PUSH
- SW0:0, SW0:1, SW0:10, SW0:11, SW0:12, SW0:13, SW0:14, SW0:15, SW0:2, SW0:3, SW0:4, SW0:5, SW0:6, SW0:7, SW0:8, SW0:9, SW1:0, SW1:1, SW1:10, SW1:11, SW1:12, SW1:13, SW1:14, SW1:15, SW1:2, SW1:3, SW1:4, SW1:5, SW1:6, SW1:7, SW1:8, SW1:9, SW2:0, SW2:1, SW2:10, SW2:11, SW2:12, SW2:13, SW2:14, SW2:15, SW2:2, SW2:3, SW2:4, SW2:5, SW2:6, SW2:7, SW2:8, SW2:9, SW3:0, SW3:1, SW3:10, SW3:11, SW3:12, SW3:13, SW3:14, SW3:15, SW3:2, SW3:3, SW3:4, SW3:5, SW3:6, SW3:7, SW3:8, SW3:9, SW4:0, SW4:1, SW4:10, SW4:11, SW4:12, SW4:13, SW4:14, SW4:15, SW4:2, SW4:3, SW4:4, SW4:5, SW4:6, SW4:7, SW4:8, SW4:9, SW5:0, SW5:1, SW5:10, SW5:11, SW5:12, SW5:13, SW5:14, SW5:15, SW5:2, SW5:3, SW5:4, SW5:5, SW5:6, SW5:7, SW5:8, SW5:9, SW6:0, SW6:1, SW6:10, SW6:11, SW6:12, SW6:13, SW6:14, SW6:15, SW6:2, SW6:3, SW6:4, SW6:5, SW6:6, SW6:7, SW6:8, SW6:9, SW7:0, SW7:1, SW7:2, SW7:3: footprint Keyboard:CHERRY_PCB_100H_With_led -> Keyboard:CHERRY_PCB_100H_With_led2
Connections:
- net labels added: VCC

Commit message: 3° commit
Connections:
- net labels removed: VCC
- wire segments 972 -> 745

Commit message: 4o step
Connections:
- net GND: now also U1.1 (GND)
- removed net LED_MATRIX_ANODE: SW0:0.3, SW0:1.3, SW0:10.3, SW0:11.3, SW0:12.3, SW0:13.3, SW0:14.3, SW0:15.3, SW0:2.3, SW0:3.3, SW0:4.3, SW0:5.3, SW0:6.3, SW0:7.3, SW0:8.3, SW0:9.3, SW1:0.3, SW1:1.3, SW1:10.3, SW1:11.3, SW1:12.3, SW1:13.3, SW1:14.3, SW1:15.3, SW1:2.3, SW1:3.3, SW1:4.3, SW1:5.3, SW1:6.3, SW1:7.3, SW1:8.3, SW1:9.3, SW2:0.3, SW2:1.3, SW2:10.3, SW2:11.3, SW2:12.3, SW2:13.3, SW2:14.3, SW2:15.3, SW2:2.3, SW2:3.3, SW2:4.3, SW2:5.3, SW2:6.3, SW2:7.3, SW2:8.3, SW2:9.3, SW3:0.3, SW3:1.3, SW3:10.3, SW3:11.3, SW3:12.3, SW3:13.3, SW3:14.3, SW3:15.3, SW3:2.3, SW3:3.3, SW3:4.3, SW3:5.3, SW3:6.3, SW3:7.3, SW3:8.3, SW3:9.3, SW4:0.3, SW4:1.3, SW4:10.3, SW4:11.3, SW4:12.3, SW4:13.3, SW4:14.3, SW4:15.3, SW4:2.3, SW4:3.3, SW4:4.3, SW4:5.3, SW4:6.3, SW4:7.3, SW4:8.3, SW4:9.3, SW5:0.3, SW5:1.3, SW5:10.3, SW5:11.3, SW5:12.3, SW5:13.3, SW5:14.3, SW5:15.3, SW5:2.3, SW5:3.3, SW5:4.3, SW5:5.3, SW5:6.3, SW5:7.3, SW5:8.3, SW5:9.3, SW6:0.3, SW6:1.3, SW6:10.3, SW6:11.3, SW6:12.3, SW6:13.3, SW6:14.3, SW6:15.3, SW6:2.3, SW6:3.3, SW6:4.3, SW6:5.3, SW6:6.3, SW6:7.3, SW6:8.3, SW6:9.3, SW7:0.3, SW7:1.3, SW7:2.3, SW7:3.3
- removed net LED_MATRIX_KATODE: SW0:0.4, SW0:1.4, SW0:10.4, SW0:11.4, SW0:12.4, SW0:13.4, SW0:14.4, SW0:15.4, SW0:2.4, SW0:3.4, SW0:4.4, SW0:5.4, SW0:6.4, SW0:7.4, SW0:8.4, SW0:9.4, SW1:0.4, SW1:1.4, SW1:10.4, SW1:11.4, SW1:12.4, SW1:13.4, SW1:14.4, SW1:15.4, SW1:2.4, SW1:3.4, SW1:4.4, SW1:5.4, SW1:6.4, SW1:7.4, SW1:8.4, SW1:9.4, SW2:0.4, SW2:1.4, SW2:10.4, SW2:11.4, SW2:12.4, SW2:13.4, SW2:14.4, SW2:15.4, SW2:2.4, SW2:3.4, SW2:4.4, SW2:5.4, SW2:6.4, SW2:7.4, SW2:8.4, SW2:9.4, SW3:0.4, SW3:1.4, SW3:10.4, SW3:11.4, SW3:12.4, SW3:13.4, SW3:14.4, SW3:15.4, SW3:2.4, SW3:3.4, SW3:4.4, SW3:5.4, SW3:6.4, SW3:7.4, SW3:8.4, SW3:9.4, SW4:0.4, SW4:1.4, SW4:10.4, SW4:11.4, SW4:12.4, SW4:13.4, SW4:14.4, SW4:15.4, SW4:2.4, SW4:3.4, SW4:4.4, SW4:5.4, SW4:6.4, SW4:7.4, SW4:8.4, SW4:9.4, SW5:0.4, SW5:1.4, SW5:10.4, SW5:11.4, SW5:12.4, SW5:13.4, SW5:14.4, SW5:15.4, SW5:2.4, SW5:3.4, SW5:4.4, SW5:5.4, SW5:6.4, SW5:7.4, SW5:8.4, SW5:9.4, SW6:0.4, SW6:1.4, SW6:10.4, SW6:11.4, SW6:12.4, SW6:13.4, SW6:14.4, SW6:15.4, SW6:2.4, SW6:3.4, SW6:4.4, SW6:5.4, SW6:6.4, SW6:7.4, SW6:8.4, SW6:9.4, SW7:0.4, SW7:1.4, SW7:2.4, SW7:3.4

Commit message: 5o step
Connections:
- net ROW4: now also SW7:4.1, SW7:5.1
- net at D4:2.1 (A), SW4:2.2: now also SW7:4.2, SW7:5.2
Other:
- moved on the sheet: L1, L2, L3, R1, R2, R3, SW7:4, SW7:5
Changed lines of the file:
@@
 L GND #PWR01
 U 1 1 4F329C8B
-P 3100 5450
-F 0 "#PWR01" H 3100 5450 30  0001 C CNN
-F 1 "GND" H 3100 5380 30  0001 C CNN
-F 2 "" H 3100 5450 60  0001 C CNN
-F 3 "" H 3100 5450 60  0001 C CNN
-	1    3100 5450
+P 2050 5950
+F 0 "#PWR01" H 2050 5950 30  0001 C CNN
+F 1 "GND" H 2050 5880 30  0001 C CNN
+F 2 "" H 2050 5950 60  0001 C CNN
+F 3 "" H 2050 5950 60  0001 C CNN
+	1    2050 5950
 	0    -1   -1   0
 $EndComp
@@
 L GND #PWR02
 U 1 1 4F329C86
-P 3100 5150
-F 0 "#PWR02" H 3100 5150 30  0001 C CNN
-F 1 "GND" H 3100 5080 30  0001 C CNN
-F 2 "" H 3100 5150 60  0001 C CNN
-F 3 "" H 3100 5150 60  0001 C CNN
-	1    3100 5150
+P 2050 5650
+F 0 "#PWR02" H 2050 5650 30  0001 C CNN
+F 1 "GND" H 2050 5580 30  0001 C CNN
+F 2 "" H 2050 5650 60  0001 C CNN
+F 3 "" H 2050 5650 60  0001 C CNN
+	1    2050 5650
 	0    -1   -1   0
 $EndComp
@@
 L RESISTOR R2
 U 1 1 4E2ADB7D
-P 2400 5450
-F 0 "R2" V 2400 5450 50  0000 C CNN
-F 1 "R_B" V 2450 5450 50  0000 C CNN
-F 2 "footprints:RESISTOR" H 2400 5450 60  0001 C CNN
-F 3 "" H 2400 5450 60  0001 C CNN
-	1    2400 5450
+P 1350 5950
+F 0 "R2" V 1350 5950 50  0000 C CNN
+F 1 "R_B" V 1400 5950 50  0000 C CNN
+F 2 "footprints:RESISTOR" H 1350 5950 60  0001 C CNN
+F 3 "" H 1350 5950 60  0001 C CNN
+	1    1350 5950
 	0    1    1    0
 $EndComp
@@
 L LED L3
 U 1 1 4E07882A
-P 2850 5750
-F 0 "L3" H 2850 5850 50  0000 C CNN
-F 1 "LED_C" H 2850 5650 50  0000 C CNN
-F 2 "footprints:CHERRY_MX_LED" H 2850 5750 60  0001 C CNN
-F 3 "" H 2850 5750 60  0001 C CNN
-	1    2850 5750
+P 1800 6250
+F 0 "L3" H 1800 6350 50  0000 C CNN
+F 1 "LED_C" H 1800 6150 50  0000 C CNN
+F 2 "footprints:CHERRY_MX_LED" H 1800 6250 60  0001 C CNN
+F 3 "" H 1800 6250 60  0001 C CNN
+	1    1800 6250
 	1    0    0    -1
 $EndComp
-Text Label 2150 5750 2    60   ~ 0
+Text Label 1100 6250 2    60   ~ 0
 LED_C
-Text Label 2150 5150 2    60   ~ 0
+Text Label 1100 5650 2    60   ~ 0
 LED_A
 $Comp
 L LED L1
 U 1 1 4E035618
-P 2850 5150
-F 0 "L1" H 2850 5250 50  0000 C CNN
-F 1 "LED_A" H 2850 5050 50  0000 C CNN
-F 2 "footprints:CHERRY_MX_LED" H 2850 5150 60  0001 C CNN
-F 3 "" H 2850 5150 60  0001 C CNN
-	1    2850 5150
+P 1800 5650
+F 0 "L1" H 1800 5750 50  0000 C CNN
+F 1 "LED_A" H 1800 5550 50  0000 C CNN
+F 2 "footprints:CHERRY_MX_LED" H 1800 5650 60  0001 C CNN
+F 3 "" H 1800 5650 60  0001 C CNN
+	1    1800 5650
 	1    0    0    -1
 $EndComp
@@
 L LED L2
 U 1 1 4E035615
-P 2850 5450
-F 0 "L2" H 2850 5550 50  0000 C CNN
-F 1 "LED_B" H 2850 5350 50  0000 C CNN
-F 2 "footprints:CHERRY_MX_LED" H 2850 5450 60  0001 C CNN
-F 3 "" H 2850 5450 60  0001 C CNN
-	1    2850 5450
+P 1800 5950
+F 0 "L2" H 1800 6050 50  0000 C CNN
+F 1 "LED_B" H 1800 5850 50  0000 C CNN
+F 2 "footprints:CHERRY_MX_LED" H 1800 5950 60  0001 C CNN
+F 3 "" H 1800 5950 60  0001 C CNN
+	1    1800 5950
 	1    0    0    -1
 $EndComp
@@
 L RESISTOR R1
 U 1 1 4E03560E
-P 2400 5150
-F 0 "R1" V 2400 5150 50  0000 C CNN
-F 1 "R_A" V 2450 5150 50  0000 C CNN
-F 2 "footprints:RESISTOR" H 2400 5150 60  0001 C CNN
-F 3 "" H 2400 5150 60  0001 C CNN
-	1    2400 5150
+P 1350 5650
+F 0 "R1" V 1350 5650 50  0000 C CNN
+F 1 "R_A" V 1400 5650 50  0000 C CNN
+F 2 "footprints:RESISTOR" H 1350 5650 60  0001 C CNN
+F 3 "" H 1350 5650 60  0001 C CNN
+	1    1350 5650
 	0    1    1    0
 $EndComp
@@
 L RESISTOR R3
 U 1 1 4E03560A
-P 2400 5750
-F 0 "R3" V 2400 5750 50  0000 C CNN
-F 1 "R_C" V 2450 5750 50  0000 C CNN
-F 2 "footprints:RESISTOR" H 2400 5750 60  0001 C CNN
-F 3 "" H 2400 5750 60  0001 C CNN
-	1    2400 5750
+P 1350 6250
+F 0 "R3" V 1350 6250 50  0000 C CNN
+F 1 "R_C" V 1400 6250 50  0000 C CNN
+F 2 "footprints:RESISTOR" H 1350 6250 60  0001 C CNN
+F 3 "" H 1350 6250 60  0001 C CNN
+	1    1350 6250
 	0    1    1    0
 $EndComp
-Text Label 4650 4750 2    60   ~ 0
-ROW4
 $Comp
 L SWITCH_PUSH SW2:5
@@
 	1    0    0    -1
 $EndComp
-Text Label 2150 5450 2    60   ~ 0
+Text Label 1100 5950 2    60   ~ 0
 LED_B
 $Comp
 L GND #PWR03
 U 1 1 4FF0041A
-P 3100 5750
-F 0 "#PWR03" H 3100 5750 30  0001 C CNN
-F 1 "GND" H 3100 5680 30  0001 C CNN
-F 2 "" H 3100 5750 60  0001 C CNN
-F 3 "" H 3100 5750 60  0001 C CNN
-	1    3100 5750
+P 2050 6250
+F 0 "#PWR03" H 2050 6250 30  0001 C CNN
+F 1 "GND" H 2050 6180 30  0001 C CNN
+F 2 "" H 2050 6250 60  0001 C CNN
+F 3 "" H 2050 6250 60  0001 C CNN
+	1    2050 6250
 	0    -1   -1   0
 $EndComp
@@
 L SWITCH_PUSH SW7:4
 U 1 1 585478A9
-P 8400 7500
-F 0 "SW7:4" H 8550 7610 50  0000 C CNN
-F 1 "Fake1" H 8400 7420 50  0000 C CNN
-F 2 "Keyboard:CHERRY_PCB_100H_With_led2" H 8400 7500 60  0001 C CNN
-F 3 "" H 8400 7500 60  0001 C CNN
-	1    8400 7500
+P 3050 5000
+F 0 "SW7:4" H 3200 5110 50  0000 C CNN
+F 1 "Fake1" H 3050 4920 50  0000 C CNN
+F 2 "Keyboard:CHERRY_PCB_100H_With_led2" H 3050 5000 60  0001 C CNN
+F 3 "" H 3050 5000 60  0001 C CNN
+	1    3050 5000
 	1    0    0    -1
 $EndComp
@@
 L SWITCH_PUSH SW7:5
 U 1 1 58547F5D
-P 9200 7500
-F 0 "SW7:5" H 9350 7610 50  0000 C CNN
-F 1 "Fake2" H 9200 7420 50  0000 C CNN
-F 2 "Keyboard:CHERRY_PCB_100H_With_led2" H 9200 7500 60  0001 C CNN
-F 3 "" H 9200 7500 60  0001 C CNN
-	1    9200 7500
+P 3050 5700
+F 0 "SW7:5" H 3200 5810 50  0000 C CNN
+F 1 "Fake2" H 3050 5620 50  0000 C CNN
+F 2 "Keyboard:CHERRY_PCB_100H_With_led2" H 3050 5700 60  0001 C CNN
+F 3 "" H 3050 5700 60  0001 C CNN
+	1    3050 5700
 	1    0    0    -1
 $EndComp
@@
 	1    0    0    -1
 $EndComp
+$Comp
+L DIODE D0:0
+U 1 1 4D9C9F15
+P 5200 1900
+F 0 "D0:0" H 5200 2000 40  0000 C CNN
+F 1 "D" H 5200 1800 40  0000 C CNN
+F 2 "footprints:DIODE" H 5200 1900 60  0001 C CNN
+F 3 "" H 5200 1900 60  0001 C CNN
+	1    5200 1900
+	-1   0    0    1
+$EndComp
+$Comp
+L SWITCH_PUSH SW1:13
+U 1 1 4D92DF9E
+P 15600 2400
+F 0 "SW1:13" H 15750 2510 50  0000 C CNN
+F 1 "]" H 15600 2320 50  0000 C CNN
+F 2 "Keyboard:CHERRY_PCB_100H_With_led2" H 15600 2400 60  0001 C CNN
+F 3 "" H 15600 2400 60  0001 C CNN
+	1    15600 2400
+	1    0    0    -1
+$EndComp
+Text Label 1350 1300 0    60   ~ 0
+GND
 Wire Wire Line
 	17500 4450 17400 4450
@@
 Wire Wire Line
 	5700 4750 5700 4950
-Connection ~ 4900 4750
-Wire Wire Line
-	4900 4950 4900 4750
 Wire Wire Line
-	4650 4750 16900 4750
+	4900 4750 4900 4950
 Wire Wire Line
 	15300 4750 15300 4950
@@
 	7100 5300 7000 5300
 Wire Wire Line
-	7100 4950 7100 5300
+	7100 4650 7100 5300
 Connection ~ 6400 2750
 Wire Wire Line
@@
 	4800 5300 5000 5300
 Wire Wire Line
-	3050 5450 3100 5450
+	2050 5950 2000 5950
 Wire Wire Line
-	3050 5150 3100 5150
+	2000 5650 2050 5650
 Wire Wire Line
 	7300 7300 7300 7500
@@
 	7350 7850 7200 7850
 Connection ~ 7200 7850
-$Comp
-L DIODE D0:0
-U 1 1 4D9C9F15
-P 5200 1900
-F 0 "D0:0" H 5200 2000 40  0000 C CNN
-F 1 "D" H 5200 1800 40  0000 C CNN
-F 2 "footprints:DIODE" H 5200 1900 60  0001 C CNN
-F 3 "" H 5200 1900 60  0001 C CNN
-	1    5200 1900
-	-1   0    0    1
-$EndComp
-$Comp
-L SWITCH_PUSH SW1:13
-U 1 1 4D92DF9E
-P 15600 2400
-F 0 "SW1:13" H 15750 2510 50  0000 C CNN
-F 1 "]" H 15600 2320 50  0000 C CNN
-F 2 "Keyboard:CHERRY_PCB_100H_With_led2" H 15600 2400 60  0001 C CNN
-F 3 "" H 15600 2400 60  0001 C CNN
-	1    15600 2400
-	1    0    0    -1
-$EndComp
-Text Label 1350 1300 0    60   ~ 0
-GND
 Wire Wire Line
-	3100 4950 3100 5750
-Connection ~ 3100 5450
+	2050 5450 2050 6250
+Connection ~ 2050 5950
 Wire Wire Line
 	1550 1300 1150 1300
 Wire Wire Line
-	1150 1300 1150 4950
+	1150 1300 1150 5450
+Connection ~ 2050 5650
+Wire Wire Line
+	1150 5450 2050 5450
+Wire Wire Line
+	3350 5000 3350 5700
+Wire Wire Line
+	3350 5700 3700 5700
+Wire Wire Line
+	3700 5700 3700 4650
+Wire Wire Line
+	3700 4650 7100 4650
+Connection ~ 7100 4950
+Wire Wire Line
+	2750 5000 2750 6050
+Wire Wire Line
+	4050 4750 16900 4750
+Text Label 4650 4750 2    60   ~ 0
+ROW4
+Connection ~ 2750 5000
+Connection ~ 4900 4750
+Wire Wire Line
+	4050 4750 4050 6050
 Wire Wire Line
-	1150 4950 3100 4950
-Connection ~ 3100 5150
+	4050 6050 2750 6050
+Connection ~ 2750 5700
 $EndSCHEMATC
