File: scdm_kicad_4_pcb.kicad_pcb (KiCad board)
At the start: 2 copper layers, 243 parts, among them SW0:0 ESC, SW0:1 1, SW0:10 0, SW0:11 -, SW0:12 =, SW0:13 BCKSPC, SW0:14 INS, SW0:15 HOME, SW0:2 2, SW0:3 3, SW0:4 4, SW0:5 5, SW0:6 6, SW0:7 7, SW0:8 8, SW0:9 9, SW1:0 PAGE_UP, SW1:1 TAB, SW1:10 O, SW1:11 P, SW1:12 [, SW1:13 ], SW1:14 \, SW1:15 DEL, SW1:2 Q, SW1:3 W, SW1:4 E, SW1:5 R, SW1:6 T, SW1:7 Y, SW1:8 U, SW1:9 I, SW2:0 END, SW2:1 PAGE_DOWN, SW2:10 K, SW2:11 L, SW2:12 ;, SW2:13 `, SW2:14 ENTER, SW2:15 LEFT, SW2:2 CAPSLOCK, SW2:3 A, SW2:4 S, SW2:5 D, SW2:6 F, SW2:7 G, SW2:8 H, SW2:9 J, SW3:0 RIGHT, SW3:1 L_SHIFT, SW3:10 ., SW3:11 /, SW3:12 R_SHIFT, SW3:13 UP, SW3:14 DOWN, SW3:15 L_CTRL, SW3:2 Z, SW3:3 X, SW3:4 C, SW3:5 V, SW3:6 B, SW3:7 N, SW3:8 M, SW3:9 ,, SW4:0 L_SUPER, SW4:1 L_ALT, SW4:10 KEYPAD_1, SW4:11 KEYPAD_2, SW4:12 KEYPAD_3, SW4:13 KEYPAD_4, SW4:14 KEYPAD_5, SW4:15 KEYPAD_6, SW4:2 SPACE, SW4:3 R_ALT, SW4:4 R_SUPER, SW4:5 MENU, SW4:6 R_CTRL, SW4:7 KEYPAD_0, SW4:8 KEYPAD_DEL, SW4:9 KEYPAD_ENTER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

Commit message: 4o step
Parts:
- moved D5:8 17.2 mm to (60.0, 145.4)
- moved D4:1 17.1 mm to (102.3, 231.3), turned to 90 degrees
- moved U1 14.1 mm to (432.4, 122.7)
- moved D6:9 12.2 mm to (98.0, 109.0), turned to 270 degrees
- moved D4:9 12.0 mm to (462.6, 221.7), turned to 90 degrees
- moved D0:1 12.0 mm to (69.9, 154.5), turned to 270 degrees
- moved D7:2 12.0 mm to (295.2, 109.2), turned to 270 degrees
- moved D1:14 12.0 mm to (309.5, 173.7), turned to 270 degrees
- moved D5:1 12.0 mm to (404.9, 173.7), turned to 90 degrees
- moved D5:3 12.0 mm to (443.3, 173.7), turned to 90 degrees
- moved D7:3 12.0 mm to (314.4, 109.3), turned to 270 degrees
- moved D0:12 12.0 mm to (281.3, 154.5), turned to 270 degrees
- moved D0:13 12.0 mm to (307.5, 154.5), turned to 270 degrees
- moved D0:7 12.0 mm to (185.1, 154.5), turned to 270 degrees
- moved D0:8 12.0 mm to (204.5, 154.5), turned to 270 degrees
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Connections:
- U1 pad 1: Net-(U1-Pad1) -> GND
Routing:
- net /COL0: track 125.9 -> 789.1 mm, vias 2 -> 6
- net /COL3: track 187.3 -> 793.9 mm, vias 6 -> 4
- net /ROW5: track 300.6 -> 905.8 mm, vias 0 -> 10
- net /COL15: track 235.9 -> 779.6 mm, vias 8 -> 4
- net /COL9: track 123.3 -> 663.1 mm, vias 3 -> 7
- net /COL2: track 187.1 -> 726.1 mm, vias 4 -> 8
- net /COL14: track 91.0 -> 621.7 mm, vias 2 -> 3
- net /COL6: track 93.7 -> 592.7 mm, vias 2 -> 6
- net /COL7: track 139.5 -> 599.5 mm, vias 2 -> 6
- net /COL4: track 93.7 -> 550.5 mm, vias 2 -> 4
- net /COL10: track 123.3 -> 574.5 mm, vias 3 -> 5
- net /COL11: track 246.3 -> 687.2 mm
- net /COL8: track 212.5 -> 641.9 mm, vias 6 -> 3
- net /COL12: track 290.2 -> 715.0 mm, vias 5 -> 2
- net /COL5: track 176.3 -> 560.4 mm, vias 7 -> 2
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Other:
- copper layers 2 -> 4

Commit message: 5o step
Connections:
- SW7:4 pad 1: Net-(SW7:4-Pad1) -> /ROW4
- SW7:4 pad 2: Net-(SW7:4-Pad2) -> Net-(D4:2-Pad1)
- SW7:5 pad 1: Net-(SW7:5-Pad1) -> /ROW4
- SW7:5 pad 2: Net-(SW7:5-Pad2) -> Net-(D4:2-Pad1)
Routing:
- net Net-(D4:2-Pad1): track 11.8 -> 89.5 mm
- net /ROW4: track 739.5 -> 751.0 mm

Commit message: 5o step con aggiunta del taglio
Other:
- board outline added: 428 x 141 mm
Changed lines of the file:
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@@
-(kicad_pcb (version 4) (host pcbnew 4.0.5-e0-6337~49~ubuntu14.04.1)
+(kicad_pcb (version 4) (host pcbnew 4.0.6-e0-6349~53~ubuntu14.04.1)
   (general
     (links 361)
     (no_connects 0)
-    (area 0 0 0 0)
+    (area 51.285883 99.749695 479.445885 296)
     (thickness 1.6002)
-    (drawings 135)
+    (drawings 149)
     (tracks 2286)
     (zones 0)
@@
     (pad "" np_thru_hole circle (at 0 0) (size 3.5 3.5) (drill 2.7) (layers *.Cu *.Mask))
   )
+  (gr_line (start 51.4 240.8) (end 51.4 99.8) (angle 90) (layer Edge.Cuts) (width 0.381))
+  (gr_line (start 128.2 240.8) (end 51.4 240.8) (angle 90) (layer Edge.Cuts) (width 0.381))
+  (gr_line (start 128.2 223.8) (end 128.2 240.8) (angle 90) (layer Edge.Cuts) (width 0.381))
+  (gr_line (start 142.4 223.8) (end 128.2 223.8) (angle 90) (layer Edge.Cuts) (width 0.381))
+  (gr_line (start 142.4 240.8) (end 142.4 223.8) (angle 90) (layer Edge.Cuts) (width 0.381))
+  (gr_line (start 226.6 240.8) (end 142.4 240.8) (angle 90) (layer Edge.Cuts) (width 0.381))
+  (gr_line (start 226.6 223.8) (end 226.6 240.8) (angle 90) (layer Edge.Cuts) (width 0.381))
+  (gr_line (start 240.6 223.8) (end 226.6 223.8) (angle 90) (layer Edge.Cuts) (width 0.381))
+  (gr_line (start 240.6 240.8) (end 240.6 223.8) (angle 90) (layer Edge.Cuts) (width 0.381))
+  (gr_line (start 479.4 240.8) (end 240.6 240.8) (angle 90) (layer Edge.Cuts) (width 0.381))
+  (gr_line (start 479.4 144.2) (end 479.4 240.8) (angle 90) (layer Edge.Cuts) (width 0.381))
+  (gr_line (start 471.4 144.2) (end 479.4 144.2) (angle 90) (layer Edge.Cuts) (width 0.381))
+  (gr_line (start 471.4 99.8) (end 471.4 144.2) (angle 90) (layer Edge.Cuts) (width 0.381))
+  (gr_line (start 51.4 99.8) (end 471.4 99.8) (angle 90) (layer Edge.Cuts) (width 0.381))
   (gr_circle (center 471.155917 168.420922) (end 472.905917 168.420922) (layer Dwgs.User) (width 0.1))
   (gr_circle (center 64.375917 230.850922) (end 66.375917 230.850922) (layer Dwgs.User) (width 0.1))
@@
   (segment (start 62 208.2) (end 62 220.78) (width 0.762) (layer In1.Cu) (net 21))
   (segment (start 63.68 206.52) (end 62 208.2) (width 0.762) (layer In1.Cu) (net 21))
-  (segment (start 210.14 225.72) (end 211.08 225.72) (width 0.762) (layer In1.Cu) (net 22) (status C00000))
-  (segment (start 211.08 225.72) (end 214.4 222.4) (width 0.762) (layer In1.Cu) (net 22) (status 400000))
+  (segment (start 210.14 225.72) (end 211.08 225.72) (width 0.762) (layer In1.Cu) (net 22))
+  (segment (start 211.08 225.72) (end 214.4 222.4) (width 0.762) (layer In1.Cu) (net 22))
   (segment (start 163.94 225.72) (end 165.08 225.72) (width 0.762) (layer In1.Cu) (net 22))
   (segment (start 165.08 225.72) (end 168.4 222.4) (width 0.762) (layer In1.Cu) (net 22))
@@
   (segment (start 102.3 229.7) (end 102.3 236.38) (width 0.762) (layer In1.Cu) (net 68))
   (segment (start 103.74 228.26) (end 102.3 229.7) (width 0.762) (layer In1.Cu) (net 68))
-  (segment (start 176 236.38) (end 176 236.6) (width 0.762) (layer In1.Cu) (net 69) (status C00000))
-  (segment (start 176 236.6) (end 177.6 238.2) (width 0.762) (layer In1.Cu) (net 69) (status 400000))
-  (segment (start 199.94 228.26) (end 203.79 228.26) (width 0.762) (layer In1.Cu) (net 69) (status 800000))
+  (segment (start 176 236.38) (end 176 236.6) (width 0.762) (layer In1.Cu) (net 69))
+  (segment (start 176 236.6) (end 177.6 238.2) (width 0.762) (layer In1.Cu) (net 69))
+  (segment (start 199.94 228.26) (end 203.79 228.26) (width 0.762) (layer In1.Cu) (net 69))
   (segment (start 199.4 228.8) (end 199.94 228.26) (width 0.762) (layer In1.Cu) (net 69))
   (segment (start 199.4 236.6) (end 199.4 228.8) (width 0.762) (layer In1.Cu) (net 69))
   (segment (start 197.8 238.2) (end 199.4 236.6) (width 0.762) (layer In1.Cu) (net 69))
   (segment (start 177.6 238.2) (end 197.8 238.2) (width 0.762) (layer In1.Cu) (net 69))
-  (segment (start 157.59 228.26) (end 152.54 228.26) (width 0.762) (layer In1.Cu) (net 69) (status 400000))
-  (segment (start 174.18 238.2) (end 176 236.38) (width 0.762) (layer In1.Cu) (net 69) (status 800000))
+  (segment (start 157.59 228.26) (end 152.54 228.26) (width 0.762) (layer In1.Cu) (net 69))
+  (segment (start 174.18 238.2) (end 176 236.38) (width 0.762) (layer In1.Cu) (net 69))
   (segment (start 152.2 238.2) (end 174.18 238.2) (width 0.762) (layer In1.Cu) (net 69))
   (segment (start 151.4 237.4) (end 152.2 238.2) (width 0.762) (layer In1.Cu) (net 69))

Commit message: 5o step con aggiunta del taglio
Other:
- board text added: "Wondersys Srl"
Changed lines of the file:
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@@
     (links 361)
     (no_connects 0)
-    (area 51.285883 99.749695 479.445885 296)
+    (area 51.209499 99.609499 479.590501 240.990501)
     (thickness 1.6002)
-    (drawings 149)
+    (drawings 150)
     (tracks 2286)
     (zones 0)
@@
     (pad "" np_thru_hole circle (at 0 0) (size 3.5 3.5) (drill 2.7) (layers *.Cu *.Mask))
   )
+  (gr_text "Wondersys Srl" (at 342 191) (layer F.Adhes)
+    (effects (font (size 4 3) (thickness 0.3048) italic))
+  )
   (gr_line (start 51.4 240.8) (end 51.4 99.8) (angle 90) (layer Edge.Cuts) (width 0.381))
